File: link-poe/link-poe.kicad_pcb (KiCad board)
At the start: 4 copper layers, 72 x 22 mm, 41 parts, among them J101 2x05_Horizontal, J102 NE8FAH, J103 DX07S016JA3, J104 2x05_Horizontal, J105 NE8FAH, J106 WAGO 2065-100, J107 WAGO 2065-100, J108 WAGO 2065-100, J109 WAGO 2065-100, Q301 BSC010N04LS, Q302 BSC010N04LS, U301 LM74502-Q1, U501 TPSM33625

Commit message: Update Library
Parts:
- C503, C504: value 22u -> 10u

Commit message: Replace step-down
Parts:
- removed R501: 40k2, V2_Resistor_SMD:R_0603
- removed R502: 10k, V2_Resistor_SMD:R_0603
- C503, C504: value 10u -> 22u
- U501: value TPSM33625 -> TPSM33620S5QRDNRQ1
Connections:
- net +VBUS renamed /+VBUS
- net +VLINK renamed /+VLINK
- net Shield renamed /Shield
- U501 pad 11: /Power +5V/Vcc -> GND
- U501 pad 9: /Power +5V/Feedback -> +5V
Routing:
- net +5V: track 0.68 -> 14.7 mm, vias 11 -> 10
- net /Power +5V/Vcc: track 9.70 -> 1.64 mm
- net /Power +5V/Feedback: track 3.13 -> 0.00 mm
- net GND: track 14.2 -> 11.9 mm, vias 50 -> 48

Commit message: Update
Parts:
- renumbered C505 to C503, C503 to C504, C504 to C505, ICON102 to ICON101, ICON101 to ICON102, ICON106 to ICON105, ICON105 to ICON106, INFO102 to INFO101, INFO101 to INFO102, J102 to J101, J105 to J102, J106 to J103, J108 to J104, J101 to J105, J104 to J106, J109 to J108, J103 to J109

Commit message: Refresh
Parts:
- C301, C302, C502, C503: footprint V2_Capacitor_SMD:C_0603 -> V2_Capacitor_SMD:C_1608
- C501, C504, C505: footprint V2_Capacitor_SMD:C_1210 -> V2_Capacitor_SMD:C_3225
- INFO102: value Layer_Numbers -> Layer_Numbers-4; footprint V2_Production:Layer_Numbers -> V2_Production:Layer_Numbers-4
- R101, R102, R301, R302: footprint V2_Resistor_SMD:R_0603 -> V2_Resistor_SMD:R_1608
Connections:
- J109 pad V: /+VBUS -> unconnected-(J109-VBUS-PadV)
Routing:
- net /+VBUS: track 8.27 -> 0.00 mm, vias 2 -> 0
