File: link-poe/PolarityProtection.kicad_sch (KiCad schematic)
At the start: 6 parts, among them Q301 BSC010N04LS, Q302 BSC010N04LS, U301 LM74502-Q1

Commit message: Update
Changed lines of the file:
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@@
 	(wire
 		(pts
-			(xy 102.87 86.36) (xy 121.92 86.36)
+			(xy 101.6 86.36) (xy 121.92 86.36)
 		)
 		(stroke
@@
 	(wire
 		(pts
-			(xy 176.53 86.36) (xy 194.31 86.36)
+			(xy 176.53 86.36) (xy 195.58 86.36)
 		)
 		(stroke
@@
 	(hierarchical_label "Input"
 		(shape input)
-		(at 102.87 86.36 180)
+		(at 101.6 86.36 180)
 		(effects
 			(font
@@
 	(hierarchical_label "Output"
 		(shape output)
-		(at 194.31 86.36 0)
+		(at 195.58 86.36 0)
 		(effects
 			(font

Commit message: Update usb + link-poe
Parts:
- C301: footprint Capacitor_SMD:C_0603_1608Metric -> V2_Capacitor_SMD:C_0603; symbol Device:C_Small -> V2_Device:C_0603_0u22; Mouser (none) -> 603-CC0603JRX79BB224
- Q301, Q302: Mouser (none) -> 726-BSC010N04LS
- R301: footprint Resistor_SMD:R_0603_1608Metric -> V2_Resistor_SMD:R_0603; symbol Device:R_Small -> V2_Device:R_0603_100k; Mouser (none) -> 71-CRCW0603100KFKEAC
- R302: footprint Resistor_SMD:R_0603_1608Metric -> V2_Resistor_SMD:R_0603; symbol Device:R_Small -> V2_Device:R_0603_3k9; Mouser (none) -> 71-CRCW06033K90FKEAC
- U301: Mouser (none) -> 595-LM74502HQDDFRQ1
Changed lines of the file:
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@@
+			)
+		)
+		(property "Mouser" "726-BSC010N04LS"
+			(at 166.878 88.9 0)
+			(effects
+				(font
+					(size 1.27 1.27)
+				)
+				(hide yes)
 			)
 		)
@@
 			)
 		)
+		(property "Mouser" "595-LM74502HQDDFRQ1"
+			(at 151.13 106.68 0)
+			(effects
+				(font
+					(size 1.27 1.27)
+				)
+				(hide yes)
+			)
+		)
 		(pin "1"
 		)
@@
 	)
 	(symbol
-		(lib_id "Device:R_Small")
+		(lib_id "V2_Device:R_0603_100k")
 		(at 121.92 111.76 0)
 		(unit 1)
@@
 		)
 		(property "Value" "100k"
-			(at 114.3 113.03 0)
-			(effects
-				(font
-					(size 1.27 1.27)
-				)
-				(justify left)
-			)
-		)
-		(property "Footprint" "Resistor_SMD:R_0603_1608Metric"
+			(at 116.586 112.776 0)
+			(effects
+				(font
+					(size 1.27 1.27)
+				)
+			)
+		)
+		(property "Footprint" "V2_Resistor_SMD:R_0603"
+			(at 121.92 127.508 0)
+			(effects
+				(font
+					(size 1.27 1.27)
+				)
+				(hide yes)
+			)
+		)
+		(property "Datasheet" ""
 			(at 121.92 111.76 0)
 			(effects
@@
 			)
 		)
-		(property "Datasheet" "~"
-			(at 121.92 111.76 0)
-			(effects
-				(font
-					(size 1.27 1.27)
-				)
-				(hide yes)
-			)
-		)
 		(property "Description" "Resistor, small symbol"
-			(at 121.92 111.76 0)
+			(at 121.92 123.952 0)
+			(effects
+				(font
+					(size 1.27 1.27)
+				)
+				(hide yes)
+			)
+		)
+		(property "Mouser" "71-CRCW0603100KFKEAC"
+			(at 121.92 127.254 0)
 			(effects
 				(font
@@
 	)
 	(symbol
-		(lib_id "Device:C_Small")
+		(lib_id "V2_Device:C_0603_0u22")
 		(at 135.89 101.6 0)
 		(unit 1)
@@
 		)
 		(property "Value" "0u22"
-			(at 128.27 102.87 0)
-			(effects
-				(font
-					(size 1.27 1.27)
-				)
-				(justify left)
-			)
-		)
-		(property "Footprint" "Capacitor_SMD:C_0603_1608Metric"
+			(at 128.27 102.616 0)
+			(effects
+				(font
+					(size 1.27 1.27)
+				)
+				(justify left)
+			)
+		)
+		(property "Footprint" "V2_Capacitor_SMD:C_0603"
+			(at 135.89 118.618 0)
+			(effects
+				(font
+					(size 1.27 1.27)
+				)
+				(hide yes)
+			)
+		)
+		(property "Datasheet" ""
 			(at 135.89 101.6 0)
 			(effects
@@
 			)
 		)
-		(property "Datasheet" "~"
-			(at 135.89 101.6 0)
-			(effects
-				(font
-					(size 1.27 1.27)
-				)
-				(hide yes)
-			)
-		)
 		(property "Description" "Unpolarized capacitor, small symbol"
-			(at 135.89 101.6 0)
+			(at 135.89 115.062 0)
+			(effects
+				(font
+					(size 1.27 1.27)
+				)
+				(hide yes)
+			)
+		)
+		(property "Mouser" "603-CC0603JRX79BB224"
+			(at 135.89 118.618 0)
 			(effects
 				(font
@@
 	)
 	(symbol
-		(lib_id "Device:R_Small")
+		(lib_id "V2_Device:R_0603_3k9")
 		(at 121.92 116.84 0)
 		(unit 1)
@@
 		(dnp no)
 		(property "Reference" "R302"
-			(at 114.3 115.57 0)
+			(at 114.3 116.078 0)
 			(effects
 				(font
@@
 		)
 		(property "Value" "3k9"
-			(at 114.3 118.11 0)
-			(effects
-				(font
-					(size 1.27 1.27)
-				)
-				(justify left)
-			)
-		)
-		(property "Footprint" "Resistor_SMD:R_0603_1608Metric"
+			(at 116.078 118.364 0)
+			(effects
+				(font
+					(size 1.27 1.27)
+				)
+			)
+		)
+		(property "Footprint" "V2_Resistor_SMD:R_0603"
+			(at 121.92 132.588 0)
+			(effects
+				(font
+					(size 1.27 1.27)
+				)
+				(hide yes)
+			)
+		)
+		(property "Datasheet" ""
 			(at 121.92 116.84 0)
 			(effects
@@
 			)
 		)
-		(property "Datasheet" "~"
-			(at 121.92 116.84 0)
-			(effects
-				(font
-					(size 1.27 1.27)
-				)
-				(hide yes)
-			)
-		)
 		(property "Description" "Resistor, small symbol"
-			(at 121.92 116.84 0)
+			(at 121.92 129.032 0)
+			(effects
+				(font
+					(size 1.27 1.27)
+				)
+				(hide yes)
+			)
+		)
+		(property "Mouser" "71-CRCW06033K90FKEAC"
+			(at 121.92 133.096 0)
 			(effects
 				(font
@@
 			(effects
 				(font
+					(size 1.27 1.27)
+				)
+				(hide yes)
+			)
+		)
+		(property "Mouser" "726-BSC010N04LS"
+			(at 155.702 88.9 0)
+			(effects
+				(font

Commit message: Update power symbols
Parts:
- added C301: 0u1, V2_Capacitor_SMD:C_0603, symbol V2_Device:C_0603_0u1
- renumbered C301 to C302
Connections:
- net GND: now also C301.2
- net Input: now also C301.1
Changed lines of the file:
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@@
+	)
+	(junction
+		(at 109.22 86.36)
+		(diameter 0)
+		(color 0 0 0 0)
 	)
 	(junction
@@
 	(wire
 		(pts
-			(xy 101.6 86.36) (xy 121.92 86.36)
+			(xy 101.6 86.36) (xy 109.22 86.36)
 		)
 		(stroke
@@
 		(pts
 			(xy 135.89 109.22) (xy 127 109.22)
+		)
+		(stroke
+			(width 0)
+			(type default)
+		)
+	)
+	(wire
+		(pts
+			(xy 109.22 86.36) (xy 121.92 86.36)
 		)
 		(stroke
@@
 			)
 			(justify left)
+		)
+	)
+	(symbol
+		(lib_id "V2_power:GND")
+		(at 109.22 91.44 0)
+		(unit 1)
+		(exclude_from_sim no)
+		(in_bom yes)
+		(on_board yes)
+		(dnp no)
+		(property "Reference" "#PWR0301"
+			(at 109.22 97.79 0)
+			(effects
+				(font
+					(size 1.27 1.27)
+				)
+				(hide yes)
+			)
+		)
+		(property "Value" "GND"
+			(at 109.22 95.504 0)
+			(effects
+				(font
+					(size 1.27 1.27)
+				)
+				(hide yes)
+			)
+		)
+		(property "Footprint" ""
+			(at 109.22 91.44 0)
+			(effects
+				(font
+					(size 1.27 1.27)
+				)
+				(hide yes)
+			)
+		)
+		(property "Datasheet" ""
+			(at 109.22 91.44 0)
+			(effects
+				(font
+					(size 1.27 1.27)
+				)
+				(hide yes)
+			)
+		)
+		(property "Description" "Power symbol creates a global label with name \"GND\" , ground"
+			(at 108.966 101.854 0)
+			(effects
+				(font
+					(size 1.27 1.27)
+				)
+				(hide yes)
+			)
+		)
+		(pin "1"
+		)
+		(instances
+			(project "link-poe"
+				(path "/6c8448b4-b04d-47e1-934e-e40cbe27a7be/e1a18e88-9abf-461b-8346-1c1c4b1e9326"
+					(reference "#PWR0301")
+					(unit 1)
+				)
+			)
 		)
 	)
@@
 	)
 	(symbol
+		(lib_id "V2_Device:C_0603_0u1")
+		(at 109.22 88.9 0)
+		(unit 1)
+		(exclude_from_sim no)
+		(in_bom yes)
+		(on_board yes)
+		(dnp no)
+		(property "Reference" "C301"
+			(at 111.76 87.63 0)
+			(effects
+				(font
+					(size 1.27 1.27)
+				)
+				(justify left)
+			)
+		)
+		(property "Value" "0u1"
+			(at 111.76 90.17 0)
+			(effects
+				(font
+					(size 1.27 1.27)
+				)
+				(justify left)
+			)
+		)
+		(property "Footprint" "V2_Capacitor_SMD:C_0603"
+			(at 109.22 105.918 0)
+			(effects
+				(font
+					(size 1.27 1.27)
+				)
+				(hide yes)
+			)
+		)
+		(property "Datasheet" ""
+			(at 109.22 88.9 0)
+			(effects
+				(font
+					(size 1.27 1.27)
+				)
+				(hide yes)
+			)
+		)
+		(property "Description" "Unpolarized capacitor, small symbol"
+			(at 109.22 102.362 0)
+			(effects
+				(font
+					(size 1.27 1.27)
+				)
+				(hide yes)
+			)
+		)
+		(property "Mouser" "810-CGA3E2X7R1H104MA"
+			(at 109.22 106.172 0)
+			(effects
+				(font
+					(size 1.27 1.27)
+				)
+				(hide yes)
+			)
+		)
+		(pin "1"
+		)
+		(pin "2"
+		)
+		(instances
+			(project "link-poe"
+				(path "/6c8448b4-b04d-47e1-934e-e40cbe27a7be/e1a18e88-9abf-461b-8346-1c1c4b1e9326"
+					(reference "C301")
+					(unit 1)
+				)
+			)
+		)
+	)
+	(symbol
 		(lib_id "V2_Device:C_0603_0u22")
 		(at 135.89 101.6 0)
@@
 		(on_board yes)
 		(dnp no)
-		(property "Reference" "C301"
+		(property "Reference" "C302"
 			(at 128.27 100.33 0)
 			(effects
@@
 			(project "power-rj45"
 				(path "/6c8448b4-b04d-47e1-934e-e40cbe27a7be/e1a18e88-9abf-461b-8346-1c1c4b1e9326"
-					(reference "C301")
+					(reference "C302")
 					(unit 1)
 				)
@@
 	)
 	(symbol
-		(lib_id "power:GND")
+		(lib_id "V2_power:GND")
 		(at 151.13 119.38 0)
 		(unit 1)
@@
 		(on_board yes)
 		(dnp no)
-		(property "Reference" "#PWR0302"
+		(property "Reference" "#PWR0303"
 			(at 151.13 125.73 0)
 			(effects
@@
 		)
 		(property "Value" "GND"
-			(at 149.15 124.81 0)
-			(effects
-				(font
-					(size 1.27 1.27)
-				)
-				(justify left)
+			(at 151.13 123.444 0)
+			(effects
+				(font
+					(size 1.27 1.27)
+				)
 				(hide yes)
 			)
@@
 		)
 		(property "Description" "Power symbol creates a global label with name \"GND\" , ground"
-			(at 151.13 119.38 0)
+			(at 150.876 129.794 0)
 			(effects
 				(font
@@
 			(project "power-rj45"
 				(path "/6c8448b4-b04d-47e1-934e-e40cbe27a7be/e1a18e88-9abf-461b-8346-1c1c4b1e9326"
-					(reference "#PWR0302")
+					(reference "#PWR0303")
 					(unit 1)
 				)
@@
 	)
 	(symbol
-		(lib_id "power:GND")
+		(lib_id "V2_power:GND")
 		(at 121.92 119.38 0)
 		(unit 1)
@@
 		(on_board yes)
 		(dnp no)
-		(property "Reference" "#PWR0301"
+		(property "Reference" "#PWR0302"
 			(at 121.92 125.73 0)
 			(effects
@@
 		)
 		(property "Value" "GND"
-			(at 121.92 124.46 0)
+			(at 121.92 123.444 0)
 			(effects
 				(font
@@
 		)
 		(property "Description" "Power symbol creates a global label with name \"GND\" , ground"
-			(at 121.92 119.38 0)
+			(at 121.666 129.794 0)
 			(effects
 				(font
@@
 			(project "power-rj45"
 				(path "/6c8448b4-b04d-47e1-934e-e40cbe27a7be/e1a18e88-9abf-461b-8346-1c1c4b1e9326"
-					(reference "#PWR0301")
+					(reference "#PWR0302")
 					(unit 1)
 				)

Commit message: Refresh
Parts:
- C301: Manufacturer (none) -> TDK; Product (none) -> CGA3E2X7R1H104M080AA
- C302: Manufacturer (none) -> YAGEO; Product (none) -> CC0603JRX7R9BB224
- Q301, Q302: Manufacturer (none) -> Infineon Technologies; Product (none) -> BSC010N04LS
- R301: Manufacturer (none) -> Vishay; Product (none) -> CRCW0603100KFKEAC; Rating (none) -> 100mW
- R302: Manufacturer (none) -> Vishay; Product (none) -> CRCW06033K90FKEAC; Rating (none) -> 100mW
- U301: Manufacturer (none) -> Texas Instruments; Product (none) -> LM74502HQDDFRQ1
Changed lines of the file:
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@@
+			)
+		)
+		(property "Product" "BSC010N04LS"
+			(at 171.45 88.9 0)
+			(effects
+				(font
+					(size 1.27 1.27)
+				)
+				(hide yes)
+			)
+		)
+		(property "Manufacturer" "Infineon Technologies"
+			(at 168.91 88.9 0)
+			(effects
+				(font
+					(size 1.27 1.27)
+				)
+				(hide yes)
 			)
 		)
@@
 			)
 		)
+		(property "Product" "LM74502HQDDFRQ1"
+			(at 151.13 144.78 0)
+			(effects
+				(font
+					(size 1.27 1.27)
+				)
+				(hide yes)
+			)
+		)
+		(property "Manufacturer" "Texas Instruments"
+			(at 151.13 142.24 0)
+			(effects
+				(font
+					(size 1.27 1.27)
+				)
+				(hide yes)
+			)
+		)
 		(pin "1"
 		)
@@
 			)
 		)
+		(property "Rating" "100mW"
+			(at 121.92 132.08 0)
+			(effects
+				(font
+					(size 1.27 1.27)
+				)
+				(hide yes)
+			)
+		)
+		(property "Manufacturer" "Vishay"
+			(at 121.92 127 0)
+			(effects
+				(font
+					(size 1.27 1.27)
+				)
+				(hide yes)
+			)
+		)
+		(property "Product" "CRCW0603100KFKEAC"
+			(at 121.92 129.54 0)
+			(effects
+				(font
+					(size 1.27 1.27)
+				)
+				(hide yes)
+			)
+		)
 		(pin "1"
 		)
@@
 			)
 		)
+		(property "Manufacturer" "TDK"
+			(at 109.22 104.14 0)
+			(effects
+				(font
+					(size 1.27 1.27)
+				)
+				(hide yes)
+			)
+		)
+		(property "Product" "CGA3E2X7R1H104M080AA"
+			(at 109.22 106.68 0)
+			(effects
+				(font
+					(size 1.27 1.27)
+				)
+				(hide yes)
+			)
+		)
 		(pin "1"
 		)
@@
 			)
 		)
+		(property "Product" "CC0603JRX7R9BB224"
+			(at 135.89 119.38 0)
+			(effects
+				(font
+					(size 1.27 1.27)
+				)
+				(hide yes)
+			)
+		)
+		(property "Manufacturer" "YAGEO"
+			(at 135.89 116.84 0)
+			(effects
+				(font
+					(size 1.27 1.27)
+				)
+				(hide yes)
+			)
+		)
 		(pin "1"
 		)
@@
 		(property "Mouser" "71-CRCW06033K90FKEAC"
 			(at 121.92 133.096 0)
+			(effects
+				(font
+					(size 1.27 1.27)
+				)
+				(hide yes)
+			)
+		)
+		(property "Product" "CRCW06033K90FKEAC"
+			(at 121.92 134.62 0)
+			(effects
+				(font
+					(size 1.27 1.27)
+				)
+				(hide yes)
+			)
+		)
+		(property "Manufacturer" "Vishay"
+			(at 121.92 132.08 0)
+			(effects
+				(font
+					(size 1.27 1.27)
+				)
+				(hide yes)
+			)
+		)
+		(property "Rating" "100mW"
+			(at 121.92 137.16 0)
 			(effects
 				(font
@@
 			(effects
 				(font
+					(size 1.27 1.27)
+				)
+				(hide yes)
+			)
+		)
+		(property "Product" "BSC010N04LS"
+			(at 151.13 88.9 0)
+			(effects
+				(font
+					(size 1.27 1.27)
+				)
+				(hide yes)
+			)
+		)
+		(property "Manufacturer" "Infineon Technologies"
+			(at 153.67 88.9 0)
+			(effects
+				(font

Commit message: Refresh
Parts:
- C301: Rating (none) -> 50V
- Q301, Q302: Polarity (none) -> N; Rating (none) -> 40V
Changed lines of the file:
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@@
+			)
+		)
+		(property "Rating" "40V"
+			(at 171.45 88.9 0)
+			(effects
+				(font
+					(size 1.27 1.27)
+				)
+				(hide yes)
+			)
+		)
+		(property "Polarity" "N"
+			(at 168.91 88.9 0)
+			(effects
+				(font
+					(size 1.27 1.27)
+				)
+				(hide yes)
 			)
 		)
@@
 		(property "Product" "CGA3E2X7R1H104M080AA"
 			(at 109.22 106.68 0)
+			(effects
+				(font
+					(size 1.27 1.27)
+				)
+				(hide yes)
+			)
+		)
+		(property "Rating" "50V"
+			(at 109.22 111.76 0)
 			(effects
 				(font
@@
 			(at 153.67 88.9 0)
 			(effects
+				(font
+					(size 1.27 1.27)
+				)
+				(hide yes)
+			)
+		)
+		(property "Rating" "40V"
+			(at 151.13 88.9 0)
+			(effects
+				(font
+					(size 1.27 1.27)
+				)
+				(hide yes)
+			)
+		)
+		(property "Polarity" "N"
+			(at 153.67 88.9 0)
+			(effects

Commit message: Use date as revision
Parts:
- U301: Mouser 595-LM74502HQDDFRQ1 -> 595-LM74502QDDFRQ1; Product LM74502HQDDFRQ1 -> LM74502QDDFRQ1
Changed lines of the file:
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@@
 			)
 		)
-		(property "Description" "Power symbol creates a global label with name \"GND\" , ground"
+		(property "Description" ""
 			(at 108.966 101.854 0)
 			(effects
@@
 			)
 		)
-		(property "Mouser" "595-LM74502HQDDFRQ1"
+		(property "Mouser" "595-LM74502QDDFRQ1"
 			(at 151.13 106.68 0)
 			(effects
@@
 			)
 		)
-		(property "Product" "LM74502HQDDFRQ1"
+		(property "Product" "LM74502QDDFRQ1"
 			(at 151.13 144.78 0)
 			(effects
@@
 			)
 		)
-		(property "Description" "Power symbol creates a global label with name \"GND\" , ground"
+		(property "Description" ""
 			(at 150.876 129.794 0)
 			(effects
@@
 			)
 		)
-		(property "Description" "Power symbol creates a global label with name \"GND\" , ground"
+		(property "Description" ""
 			(at 121.666 129.794 0)
 			(effects

Commit message: Update Library
Parts:
- C301: symbol V2_Device:C_0603_0u1 -> V2_Capacitor:0603_0u1
- C302: symbol V2_Device:C_0603_0u22 -> V2_Capacitor:0603_0u22
- R301: symbol V2_Device:R_0603_100k -> V2_Resistor:0603_100k
- R302: symbol V2_Device:R_0603_3k9 -> V2_Resistor:0603_3k9
Changed lines of the file:
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@@
 		(on_board yes)
 		(dnp no)
-		(property "Reference" "#PWR0301"
+		(property "Reference" "#PWR301"
 			(at 109.22 97.79 0)
 			(effects
@@
 			(project "link-poe"
 				(path "/6c8448b4-b04d-47e1-934e-e40cbe27a7be/e1a18e88-9abf-461b-8346-1c1c4b1e9326"
-					(reference "#PWR0301")
+					(reference "#PWR301")
 					(unit 1)
 				)
@@
 	)
 	(symbol
-		(lib_id "V2_Device:R_0603_100k")
+		(lib_id "V2_Resistor:0603_100k")
 		(at 121.92 111.76 0)
 		(unit 1)
@@
 	)
 	(symbol
-		(lib_id "V2_Device:C_0603_0u1")
+		(lib_id "V2_Capacitor:0603_0u1")
 		(at 109.22 88.9 0)
 		(unit 1)
@@
 	)
 	(symbol
-		(lib_id "V2_Device:C_0603_0u22")
+		(lib_id "V2_Capacitor:0603_0u22")
 		(at 135.89 101.6 0)
 		(unit 1)
@@
 	)
 	(symbol
-		(lib_id "V2_Device:R_0603_3k9")
+		(lib_id "V2_Resistor:0603_3k9")
 		(at 121.92 116.84 0)
 		(unit 1)
@@
 		(on_board yes)
 		(dnp no)
-		(property "Reference" "#PWR0303"
+		(property "Reference" "#PWR303"
 			(at 151.13 125.73 0)
 			(effects
@@
 			(project "power-rj45"
 				(path "/6c8448b4-b04d-47e1-934e-e40cbe27a7be/e1a18e88-9abf-461b-8346-1c1c4b1e9326"
-					(reference "#PWR0303")
+					(reference "#PWR303")
 					(unit 1)
 				)
@@
 		(on_board yes)
 		(dnp no)
-		(property "Reference" "#PWR0302"
+		(property "Reference" "#PWR302"
 			(at 121.92 125.73 0)
 			(effects
@@
 			(project "power-rj45"
 				(path "/6c8448b4-b04d-47e1-934e-e40cbe27a7be/e1a18e88-9abf-461b-8346-1c1c4b1e9326"
-					(reference "#PWR0302")
+					(reference "#PWR302")
 					(unit 1)
 				)
