File: power-poe/power-poe.kicad_pcb (KiCad board)
At the start: 4 copper layers, 52 x 44 mm, 12 parts, among them J1 NE8FAV, J2 NE8FAV, J3 WAGO 2604-1101, J4 WAGO 2604-1101, J5 WAGO 2604-1101, J6 WAGO 2604-1101

Commit message: Update
Parts:
- J103: renamed from J5; value WAGO 2604-1101 -> Conn_01x01; footprint V2_Connector_WAGO:2604-1101 -> V2_Connector_WAGO:2601-1101
- J104: renamed from J3; value WAGO 2604-1101 -> Conn_01x01; footprint V2_Connector_WAGO:2604-1101 -> V2_Connector_WAGO:2601-1101
- J105: renamed from J6; value WAGO 2604-1101 -> Conn_01x01; footprint V2_Connector_WAGO:2604-1101 -> V2_Connector_WAGO:2601-1101
- J106: renamed from J4; value WAGO 2604-1101 -> Conn_01x01; footprint V2_Connector_WAGO:2604-1101 -> V2_Connector_WAGO:2601-1101
- moved INFO101 20.0 mm to (143.0, 115.0)
- moved J103 1.00 mm to (135.8, 82.0)
- moved J104 1.00 mm to (135.8, 77.0)
- moved J105 1.00 mm to (150.2, 82.0)
- moved J106 1.00 mm to (150.2, 77.0)
- renumbered H3 to H101, H4 to H102, ICON3 to ICON101, ICON1 to ICON102, ICON2 to ICON103, J1 to J101, J2 to J102
Routing:
- net GND: track 0.00 -> 6.13 mm, vias 2 -> 0
- net +24V: track 0.00 -> 6.13 mm
- net /RX-A: track 34.5 -> 29.9 mm, vias 1 -> 0
- net /RX-B: track 27.7 -> 30.3 mm, vias 1 -> 0
- net /TX-Y: track 31.3 -> 29.4 mm
- net /TX-Z: track 27.1 -> 27.9 mm

Commit message: Update power symbols
Parts:
- INFO101: value ORDER-NUMBER -> Order_Number
- J103, J104, J105, J106: value Conn_01x01 -> WAGO 2601-1101
Connections:
- net /Shield renamed Shield
Changed lines of the file:
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@@
 	(net 5 "/RX-B")
 	(net 6 "/TX-Y")
-	(net 7 "/Shield")
+	(net 7 "Shield")
 	(footprint "V2_Mechanical:MountingHole_5mm"
 		(layer "F.Cu")
@@
 			)
 		)
-		(property "Description" "Mounting Hole without connection"
+		(property "Description" ""
 			(at 0 0 0)
 			(unlocked yes)
@@
 				(font
 					(size 1.27 1.27)
-					(thickness 0.15)
-				)
-			)
-		)
-		(property "Sim.Enable" "0"
-			(at 0 0 0)
-			(unlocked yes)
-			(layer "F.Fab")
-			(hide yes)
-			(effects
-				(font
-					(size 1 1)
 					(thickness 0.15)
 				)
@@
 			)
 		)
-		(property "Description" "Mounting Hole without connection"
+		(property "Description" ""
 			(at 0 0 0)
 			(unlocked yes)
@@
 				(font
 					(size 1.27 1.27)
-					(thickness 0.15)
-				)
-			)
-		)
-		(property "Sim.Enable" "0"
-			(at 0 0 0)
-			(unlocked yes)
-			(layer "F.Fab")
-			(hide yes)
-			(effects
-				(font
-					(size 1 1)
 					(thickness 0.15)
 				)
@@
 			)
 		)
-		(property "Value" "Conn_01x01"
+		(property "Value" "WAGO 2601-1101"
 			(at 0.1 -9.8 90)
 			(layer "F.SilkS")
@@
 				(font
 					(size 1.27 1.27)
-					(thickness 0.15)
-				)
-			)
-		)
-		(property "Sim.Enable" "0"
-			(at 0 0 90)
-			(unlocked yes)
-			(layer "F.Fab")
-			(hide yes)
-			(effects
-				(font
-					(size 1 1)
 					(thickness 0.15)
 				)
@@
 			(fill no)
 			(layer "F.Fab")
+		)
+		(fp_text user "${REFERENCE}"
+			(at 0 0 180)
+			(layer "F.Fab")
+			(effects
+				(font
+					(size 0.75 0.75)
+					(thickness 0.1)
+					(bold yes)
+				)
+			)
 		)
 		(pad "1" thru_hole circle
@@
 				(font
 					(size 1.27 1.27)
-					(thickness 0.15)
-				)
-			)
-		)
-		(property "Sim.Enable" "0"
-			(at 0 0 90)
-			(unlocked yes)
-			(layer "F.Fab")
-			(hide yes)
-			(effects
-				(font
-					(size 1 1)
 					(thickness 0.15)
 				)
@@
 			)
 		)
-		(property "Sim.Enable" "0"
-			(at 0 0 0)
-			(unlocked yes)
-			(layer "F.Fab")
-			(hide yes)
-			(effects
-				(font
-					(size 1 1)
-					(thickness 0.15)
-				)
-			)
-		)
 		(sheetname "/")
 		(sheetfile "power-poe.kicad_sch")
@@
 			(layer "F.Fab")
 		)
+		(fp_text user "${REFERENCE}"
+			(at 0 0 0)
+			(layer "F.Fab")
+			(effects
+				(font
+					(size 0.75 0.75)
+					(thickness 0.1)
+				)
+			)
+		)
 		(pad "" np_thru_hole circle
 			(at -8.425 0)
@@
 			(keep_end_layers yes)
 			(zone_layer_connections)
-			(net 7 "/Shield")
+			(net 7 "Shield")
 			(pintype "passive")
 		)
@@
 			)
 		)
-		(property "Value" "Conn_01x01"
+		(property "Value" "WAGO 2601-1101"
 			(at 0.1 -9.8 90)
 			(layer "F.SilkS")
@@
 				(font
 					(size 1.27 1.27)
-					(thickness 0.15)
-				)
-			)
-		)
-		(property "Sim.Enable" "0"
-			(at 0 0 90)
-			(unlocked yes)
-			(layer "F.Fab")
-			(hide yes)
-			(effects
-				(font
-					(size 1 1)
 					(thickness 0.15)
 				)
@@
 			(fill no)
 			(layer "F.Fab")
+		)
+		(fp_text user "${REFERENCE}"
+			(at 0 0 180)
+			(layer "F.Fab")
+			(effects
+				(font
+					(size 0.75 0.75)
+					(thickness 0.1)
+					(bold yes)
+				)
+			)
 		)
 		(pad "1" thru_hole circle
@@
 			)
 		)
-		(property "Sim.Enable" "0"
-			(at 0 0 0)
-			(unlocked yes)
-			(layer "F.Fab")
-			(hide yes)
-			(effects
-				(font
-					(size 1 1)
-					(thickness 0.15)
-				)
-			)
-		)
 		(sheetname "/")
 		(sheetfile "power-poe.kicad_sch")
@@
 			(layer "F.Fab")
 		)
+		(fp_text user "${REFERENCE}"
+			(at 0 0 0)
+			(layer "F.Fab")
+			(effects
+				(font
+					(size 0.75 0.75)
+					(thickness 0.1)
+				)
+			)
+		)
 		(pad "" np_thru_hole circle
 			(at -8.425 0)
@@
 			(keep_end_layers yes)
 			(zone_layer_connections)
-			(net 7 "/Shield")
+			(net 7 "Shield")
 			(pintype "passive")
 		)
@@
 			)
 		)
-		(property "Value" "Conn_01x01"
+		(property "Value" "WAGO 2601-1101"
 			(at 0.1 -9.8 270)
 			(layer "F.SilkS")
@@
 				(font
 					(size 1.27 1.27)
-					(thickness 0.15)
-				)
-			)
-		)
-		(property "Sim.Enable" "0"
-			(at 0 0 270)
-			(unlocked yes)
-			(layer "F.Fab")
-			(hide yes)
-			(effects
-				(font
-					(size 1 1)
 					(thickness 0.15)
 				)
@@
 			(fill no)
 			(layer "F.Fab")
+		)
+		(fp_text user "${REFERENCE}"
+			(at 0 0 0)
+			(layer "F.Fab")
+			(effects
+				(font
+					(size 0.75 0.75)
+					(thickness 0.1)
+					(bold yes)
+				)
+			)
 		)
 		(pad "1" thru_hole circle
@@
 			)
 		)
-		(property "Value" "Conn_01x01"
+		(property "Value" "WAGO 2601-1101"
 			(at 0.1 -9.8 270)
 			(layer "F.SilkS")
@@
 				(font
 					(size 1.27 1.27)
-					(thickness 0.15)
-				)
-			)
-		)
-		(property "Sim.Enable" "0"
-			(at 0 0 270)
-			(unlocked yes)
-			(layer "F.Fab")
-			(hide yes)
-			(effects
-				(font
-					(size 1 1)
 					(thickness 0.15)
 				)
@@
 			(fill no)
 			(layer "F.Fab")
+		)
+		(fp_text user "${REFERENCE}"
+			(at 0 0 0)
+			(layer "F.Fab")
+			(effects
+				(font
+					(size 0.75 0.75)
+					(thickness 0.1)
+					(bold yes)
+				)
+			)
 		)
 		(pad "1" thru_hole circle
@@
 				(font
 					(size 1.27 1.27)
-					(thickness 0.15)
-				)
-			)
-		)
-		(property "Sim.Enable" "0"
-			(at 0 0 0)
-			(unlocked yes)
-			(layer "F.Fab")
-			(hide yes)
-			(effects
-				(font
-					(size 1 1)
 					(thickness 0.15)
 				)
@@
 			)
 		)
-		(property "Sim.Enable" "0"
-			(at 0 0 0)
-			(unlocked yes)
-			(layer "F.Fab")
-			(hide yes)
-			(effects
-				(font
-					(size 1 1)
-					(thickness 0.15)
-				)
-			)
-		)
 		(sheetname "/")
 		(sheetfile "power-poe.kicad_sch")
@@
 			)
 		)
-		(property "Value" "ORDER-NUMBER"
+		(property "Value" "Order_Number"
 			(at 0 -2.27 0)
 			(unlocked yes)
@@
 		)
 		(property "Datasheet" ""
-			(at 0 0 180)
+			(at 0 0 0)
 			(unlocked yes)
 			(layer "B.Fab")
@@
 					(thickness 0.15)
 				)
+				(justify mirror)
 			)
 		)
 		(property "Description" ""
-			(at 0 0 180)
+			(at 0 0 0)
 			(unlocked yes)
 			(layer "B.Fab")
@@
 					(thickness 0.15)
 				)
-			)
-		)
-		(property "exclude_from_bom" ""
-			(at 0 0 0)
-			(layer "B.Fab")
-			(hide yes)
-			(effects
-				(font
-					(size 1 1)
-					(thickness 0.15)
-				)
-				(justify mirror)
-			)
-		)
-		(property "Sim.Enable" "0"
-			(at 0 0 0)
-			(unlocked yes)
-			(layer "B.Fab")
-			(hide yes)
-			(effects
-				(font
-					(size 1 1)
-					(thickness 0.15)
-				)
