File: power-poe/power-poe.kicad_sch (KiCad schematic)
At the start: 12 parts, among them J1 NE8FAV, J2 NE8FAV, J3 WAGO 2604-1101, J4 WAGO 2604-1101, J5 WAGO 2604-1101, J6 WAGO 2604-1101

Commit message: Update
Parts:
- J103: renamed from J5; value WAGO 2604-1101 -> Conn_01x01; footprint V2_Connector_WAGO:2604-1101 -> V2_Connector_WAGO:2601-1101; symbol V2_Connector_WAGO:2604-1101 -> V2_Connector_WAGO:2601-1101
- J104: renamed from J3; value WAGO 2604-1101 -> Conn_01x01; footprint V2_Connector_WAGO:2604-1101 -> V2_Connector_WAGO:2601-1101; symbol V2_Connector_WAGO:2604-1101 -> V2_Connector_WAGO:2601-1101
- J105: renamed from J6; value WAGO 2604-1101 -> Conn_01x01; footprint V2_Connector_WAGO:2604-1101 -> V2_Connector_WAGO:2601-1101; symbol V2_Connector_WAGO:2604-1101 -> V2_Connector_WAGO:2601-1101
- J106: renamed from J4; value WAGO 2604-1101 -> Conn_01x01; footprint V2_Connector_WAGO:2604-1101 -> V2_Connector_WAGO:2601-1101; symbol V2_Connector_WAGO:2604-1101 -> V2_Connector_WAGO:2601-1101
- renumbered H3 to H101, H4 to H102, ICON3 to ICON101, ICON1 to ICON102, ICON2 to ICON103, J1 to J101, J2 to J102
Other:
- note added: "PoE Passive +24V IEEE 802.3af Mode B"
- moved on the sheet: H101, H102, ICON102, ICON103, J101, J102, J103, J104, J105, J106

Commit message: Update power symbols
Parts:
- INFO101: value ORDER-NUMBER -> Order_Number
- J101, J102: Mouser (none) -> 568-NE8FAV-SD
- J103, J104, J105, J106: value Conn_01x01 -> WAGO 2601-1101
Other:
- moved on the sheet: J101, J102, J103, J104, J105, J106

Commit message: Refresh
Parts:
- J101, J102: Manufacturer (none) -> Neutrik; Product (none) -> NE8FAV-SD
- J103, J104, J105, J106: Manufacturer (none) -> WAGO; Product (none) -> 2601-1101
Changed lines of the file:
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@@
+			)
+		)
+		(property "Manufacturer" "WAGO"
+			(at 128.27 147.32 0)
+			(effects
+				(font
+					(size 1.27 1.27)
+				)
+				(hide yes)
+			)
+		)
+		(property "Product" "2601-1101"
+			(at 128.27 150.368 0)
+			(effects
+				(font
+					(size 1.27 1.27)
+				)
+				(hide yes)
 			)
 		)
@@
 			)
 		)
+		(property "Manufacturer" "WAGO"
+			(at 163.83 147.32 0)
+			(effects
+				(font
+					(size 1.27 1.27)
+				)
+				(hide yes)
+			)
+		)
+		(property "Product" "2601-1101"
+			(at 163.83 150.368 0)
+			(effects
+				(font
+					(size 1.27 1.27)
+				)
+				(hide yes)
+			)
+		)
 		(pin "1"
 		)
@@
 		(property "Description" ""
 			(at 163.83 143.51 0)
+			(effects
+				(font
+					(size 1.27 1.27)
+				)
+				(hide yes)
+			)
+		)
+		(property "Manufacturer" "WAGO"
+			(at 163.83 154.94 0)
+			(effects
+				(font
+					(size 1.27 1.27)
+				)
+				(hide yes)
+			)
+		)
+		(property "Product" "2601-1101"
+			(at 163.83 157.988 0)
 			(effects
 				(font
@@
 			)
 		)
+		(property "Manufacturer" "Neutrik"
+			(at 165.1 105.41 0)
+			(effects
+				(font
+					(size 1.27 1.27)
+				)
+				(hide yes)
+			)
+		)
+		(property "Product" "NE8FAV-SD"
+			(at 165.1 107.95 0)
+			(effects
+				(font
+					(size 1.27 1.27)
+				)
+				(hide yes)
+			)
+		)
 		(pin "1"
 		)
@@
 			)
 		)
+		(property "Manufacturer" "WAGO"
+			(at 128.27 154.94 0)
+			(effects
+				(font
+					(size 1.27 1.27)
+				)
+				(hide yes)
+			)
+		)
+		(property "Product" "2601-1101"
+			(at 128.27 157.988 0)
+			(effects
+				(font
+					(size 1.27 1.27)
+				)
+				(hide yes)
+			)
+		)
 		(pin "1"
 		)
@@
 			(effects
 				(font
+					(size 1.27 1.27)
+				)
+				(hide yes)
+			)
+		)
+		(property "Manufacturer" "Neutrik"
+			(at 119.38 105.41 0)
+			(effects
+				(font
+					(size 1.27 1.27)
+				)
+				(hide yes)
+			)
+		)
+		(property "Product" "NE8FAV-SD"
+			(at 119.38 107.95 0)
+			(effects
+				(font
