File: power-link-usb/power-link-usb.kicad_pcb (KiCad board)
At the start: 4 copper layers, 60 x 30 mm, 35 parts, among them J101 NE8FAH, J102 NE8FAH, J103 DX07S016JA3, Q101 BSC010N04LS, Q102 BSC010N04LS, U101 CYPD3176-24LQ

Commit message: Fix WAGOs
Parts:
- removed R111: 5k1, V2_Resistor_SMD:R_0603
- removed R112: 1k, V2_Resistor_SMD:R_0603
- added R114: 5k1, V2_Resistor_SMD:R_0603, F.Cu at (146.8, 95.8)
- added R115: 1k, V2_Resistor_SMD:R_0603, F.Cu at (146.8, 97.2)
- moved C105 34.4 mm to (125.2, 91.0)
- moved INFO101 28.7 mm to (142.0, 115.5)
- moved C101 10.0 mm to (140.0, 109.8)
- moved C102 10.0 mm to (140.0, 111.2)
- moved C107 10.0 mm to (154.0, 87.0)
- moved J102 10.0 mm to (167.0, 99.8)
- moved Q101 10.0 mm to (153.0, 110.8)
- moved Q102 10.0 mm to (145.8, 110.8)
- moved R101 10.0 mm to (140.0, 108.2)
- moved R102 10.0 mm to (140.0, 106.5)
- moved R103 10.0 mm to (140.0, 112.8)
- moved R109 10.0 mm to (136.5, 111.2)
- moved R110 10.0 mm to (134.5, 111.2)
- moved R113 10.0 mm to (155.8, 101.5)
- moved TP101 10.0 mm to (136.2, 108.8)
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Connections:
- U101 pad 16: /Current-Min -> PGND
- U101 pad 17: PGND -> /Current-Min
Other:
- board size 60 x 30 mm -> 50 x 34.5 mm

Commit message: Update power-link-usb
Parts:
- removed the C105 at (125.2, 91.0)
- removed the C106 at (157.0, 90.8)
- removed R106, R108, R115: 1k, V2_Resistor_SMD:R_0603
- removed R107, R114: 5k1, V2_Resistor_SMD:R_0603
- removed R109, R110: 2k7, V2_Resistor_SMD:R_0603
- removed R113: 0R005, V2_Resistor_SMD:R_1210
- removed TP101, TP102, TP103: ~, V2_TestPoint:TestPoint_THTPad_D1.0mm_Drill0.5mm
- added C108: 1u, V2_Capacitor_SMD:C_0603, F.Cu at (139.2, 111.5)
- added FID101: Fiducial_Paste, V2_Fiducial:Fiducial_0.5mm_Mask1mm_Paste, F.Cu at (166.0, 116.0)
- added FID102: Fiducial_Paste, V2_Fiducial:Fiducial_0.5mm_Mask1mm_Paste, F.Cu at (118.0, 83.5)
- added FID103: Fiducial_Paste, V2_Fiducial:Fiducial_0.5mm_Mask1mm_Paste, F.Cu at (118.0, 116.0)
- added INFO102: Layer_Numbers, V2_Production:Layer_Numbers, F.Cu at (121.8, 116.2)
- added J101: 2x05_Vertical, V2_Connector_Header_1.27mm:PinHeader_2x05_P1.27mm_Vertical, B.Cu at (142.0, 86.5)
- added TVS101: SMBJ36CA, V2_Diode_SMD:D_SMB, F.Cu at (157.0, 99.5)
- added TVS102: SMBJ36CA, V2_Diode_SMD:D_SMB, F.Cu at (127.0, 99.5)
- C101: value 1u -> 10u
- C102, C103, C104: value 1u -> 0u1
- C105: renamed from C108; value 100p -> 390p
- C106: renamed from C109; value 100p -> 390p
- C107: value 100p -> 10u; footprint V2_Capacitor_SMD:C_0603 -> V2_Capacitor_SMD:C_0805
- D101: value Red -> Orange
- D102: value Orange -> Red
- R102: value 100k -> 3k9
- R103: value 1k -> 3k9
- R104: value 1k -> 330R
- R105: value 2k7 -> 330R
- U101: value CYPD3176-24LQ -> CYPM1311-48LDXI; footprint V2_Package_DFN_QFN:QFN-24-1EP_4x4mm_P0.5mm_EP2.75x2.75mm -> V2_Package_DFN_QFN:QFN-48-1EP_6x6mm_P0.4mm_EP4.6x4.6mm
- moved R103 30.1 mm to (148.8, 84.0)
- moved C107 26.8 mm to (159.2, 113.2)
- moved R102 21.6 mm to (148.8, 86.8)
- moved C101 20.8 mm to (141.8, 89.0), turned to 90 degrees
- moved R101 20.5 mm to (148.8, 89.8)
- moved C102 16.7 mm to (137.5, 94.8), turned to -90 degrees
- moved C106 13.8 mm to (148.8, 92.8)
- moved C105 9.40 mm to (148.8, 94.8)
- moved C104 5.96 mm to (143.2, 89.0), turned to -90 degrees
- moved C103 5.53 mm to (143.2, 99.2), turned to 180 degrees
- moved U101 4.03 mm to (142.0, 94.8)
- moved R104 3.61 mm to (165.5, 87.8), turned to 90 degrees
- moved R105 3.61 mm to (165.5, 94.5), turned to 90 degrees
- moved Q101 1.60 mm to (151.8, 111.8), turned to 180 degrees
- moved Q102 1.60 mm to (144.5, 111.8), turned to 0 degrees
- renumbered J103 to J102, J101 to J103, J102 to J104
Connections:
- C101 pad 1: +VBUS -> +3V3
- C101 pad 2: /Gate -> GND
- C102 pad 1: +VLINK -> +3V3
- C102 pad 2: /Gate -> GND
- C103 pad 2: PGND -> GND
- C104 pad 1: /+1V8 -> GND
- C104 pad 2: PGND -> /+1V8
- C105 pad 2: PGND -> GND
- C106 pad 2: PGND -> GND
- C107 pad 1: PGND -> +VBUS
- D101 pad 1: PGND -> Net-(D101-K)
- D101 pad 2: Net-(D101-A) -> +3V3
- D102 pad 2: +VLINK -> +3V3
- J102 pad G: PGND -> GND
- Q101 pad 1: /Source -> +VBUS
- Q101 pad 4: /Gate -> /Rail-Input
- Q101 pad 5: +VBUS -> /Drain
- Q102 pad 1: /Source -> +VLINK
- Q102 pad 4: /Gate -> /Rail-Output
- Q102 pad 5: +VLINK -> /Drain
- R101 pad 1: +VBUS -> /RESET
- R101 pad 2: /Gate -> +3V3
- R102 pad 1: /Source -> /SCK
- R102 pad 2: /Gate -> +3V3
- R103 pad 1: /Gate-Driver -> /SDA
- R103 pad 2: /Gate -> +3V3
- R104 pad 1: /Fault -> Net-(D101-K)
- R104 pad 2: Net-(D101-A) -> /LED-Orange
- R105 pad 2: GND -> /LED-Red
- U101 pad 1: /Voltage-Min -> unconnected-(U101-P3.0-Pad1)
- U101 pad 10: /Data-Mode -> /LED-Red
- U101 pad 11: +VLINK -> /LED-Orange
- U101 pad 12: /SDA -> /SWCLK
- U101 pad 13: /SCK -> /SWDIO
- U101 pad 14: /USB-CC2 -> unconnected-(U101-P1.3-Pad14)
- U101 pad 15: /USB-CC1 -> unconnected-(U101-P6.0-Pad15)
- U101 pad 16: PGND -> unconnected-(U101-P6.1-Pad16)
- U101 pad 17: /Current-Min -> unconnected-(U101-P0.0-Pad17)
- U101 pad 18: +VBUS -> unconnected-(U101-P6.2-Pad18)
- U101 pad 19: GND -> unconnected-(U101-P6.3-Pad19)
- U101 pad 2: +3V3 -> unconnected-(U101-P3.3-Pad2)
- U101 pad 22: PGND -> unconnected-(U101-P1.6-Pad22)
- U101 pad 24: /+1V8 -> +VBUS
- U101 pad 25: PGND -> +VLINK
- U101 pad 3: /Gate-Driver -> /UART-RX
- U101 pad 4: unconnected-(U101-SAFE_PWR_EN-Pad4) -> /UART-TX
- U101 pad 5: /USB+ -> +3V3
- U101 pad 6: /USB- -> GND
- U101 pad 8: /Fault -> unconnected-(U101-P5.1-Pad8)
Routing:
- net +3V3: track 0.00 -> 74.8 mm, vias 0 -> 8
- net /LED-Red: track 0.00 -> 48.9 mm, vias 0 -> 2
- net /LED-Orange: track 0.00 -> 47.6 mm, vias 0 -> 2
- net /Shield RJ45: track 0.00 -> 41.1 mm
- net /TX-Y: track 0.00 -> 36.6 mm
- net /USB-CC1: track 0.00 -> 33.9 mm, vias 0 -> 2
- net /Rail-Output: track 0.00 -> 33.4 mm, vias 0 -> 2
- net /USB-: track 0.00 -> 33.4 mm, vias 0 -> 2
- net /USB-CC2: track 0.00 -> 32.4 mm, vias 0 -> 2
- net /TX-Z: track 0.00 -> 31.6 mm
- net /USB+: track 0.00 -> 30.1 mm, vias 0 -> 2
- net /RX-A: track 0.00 -> 25.2 mm
- net +VBUS: track 0.00 -> 23.4 mm, vias 0 -> 3
- net /Rail-Input: track 0.00 -> 23.4 mm
- net /SWDIO: track 0.00 -> 18.0 mm, vias 0 -> 1
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- added copper zone on F.Cu, net +VBUS
- added copper zone on F.Cu, net +VLINK
- added copper zone on F.Cu, net /Drain
- added copper zone on F.Cu, net GND
- added copper zone on F.Cu, net Shield
- removed copper zone on B.Cu, net GND

Commit message: Refresh
Parts:
- TVS101, TVS102: value SMBJ36CA -> SMBJ33CA
Changed lines of the file:
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@@
 			)
 		)
-		(property "Value" "SMBJ36CA"
+		(property "Value" "SMBJ33CA"
 			(at 0 3.1 270)
 			(layer "F.Fab")
@@
 			)
 		)
-		(property "Value" "SMBJ36CA"
+		(property "Value" "SMBJ33CA"
 			(at 0 3.1 270)
 			(layer "F.Fab")
@@
 		(layer "F.Cu")
 		(hatch edge 0.5)
-		(priority 4)
 		(connect_pads yes
 			(clearance 0.2)
@@
 		(layer "F.Cu")
 		(hatch edge 0.5)
-		(priority 4)
 		(connect_pads yes
 			(clearance 0.2)
@@
 		(layer "F.Cu")
 		(hatch edge 0.5)
-		(priority 3)
 		(connect_pads yes
 			(clearance 0.2)
@@
 		(layer "F.Cu")
 		(hatch edge 0.508)
-		(priority 1)
 		(connect_pads yes
 			(clearance 0.2)
@@
 		(layer "F.Cu")
 		(hatch edge 0.5)
-		(priority 1)
 		(connect_pads yes
 			(clearance 0.2)
@@
 		(layer "F.Cu")
 		(hatch edge 0.5)
-		(priority 4)
 		(connect_pads yes
 			(clearance 0.2)

Commit message: Update library
Parts:
- removed J101: 2x05_Vertical, V2_Connector_Header_1.27mm:PinHeader_2x05_P1.27mm_Vertical
- added J1: >VALUE, V2_Connector_Debug:KitProg3, F.Cu at (142.0, 85.2)
