File: power-link-usb/power-link-usb.kicad_sch (KiCad schematic)
At the start: 35 parts, among them J101 NE8FAH, J102 NE8FAH, J103 DX07S016JA3, Q101 BSC010N04LS, Q102 BSC010N04LS, U101 CYPD3176-24LQ

Commit message: Fix WAGOs
Parts:
- removed R111: 5k1, V2_Resistor_SMD:R_0603, symbol V2_Device:R_0603_5k1
- removed R112: 1k, V2_Resistor_SMD:R_0603, symbol V2_Device:R_0603_1k
- added R114: 5k1, V2_Resistor_SMD:R_0603, symbol V2_Device:R_0603_5k1
- added R115: 1k, V2_Resistor_SMD:R_0603, symbol V2_Device:R_0603_1k
Connections:
- net +3V3: now also R114.1
- net Current-Min: now also U101.17 (ISNK_COARSE), R114.2, R115.1; no longer U101.16 (ISNK_FINE)
- net PGND: now also U101.16 (ISNK_FINE), R115.2; no longer U101.17 (ISNK_COARSE)
Other:
- note added: "1A"
- note added: "9-20V, Minimum 1A"
- note added: "Current Sensing The power return path between PGND and GND"
- note removed: "250mA"
- note removed: "9-20V, Minimum 250mA"
- note removed: "Current sensing Power return path between PGND and GND"
- moved on the sheet: C101, C102, C103, C104, C105, C106, C107, C108, C109, D101, D102, Q101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

Commit message: Update power-link-usb
Parts:
- removed C101, C102, C103, C104: 1u, V2_Capacitor_SMD:C_0603, symbol V2_Device:C_0603_1u
- removed C105, C106: 10u, V2_Capacitor_SMD:C_1210, symbol V2_Device:C_1210_10u
- removed C107: 100p, V2_Capacitor_SMD:C_0603, symbol V2_Device:C_0603_100p
- removed D101: Red, V2_LED:LED_0603, symbol V2_Device:LED_0603_Red
- removed D102: Orange, V2_LED:LED_0603, symbol V2_Device:LED_0603_Orange
- removed R102: 100k, V2_Resistor_SMD:R_0603, symbol V2_Device:R_0603_100k
- removed R103, R104, R106, R108, R115: 1k, V2_Resistor_SMD:R_0603, symbol V2_Device:R_0603_1k
- removed R105, R109, R110: 2k7, V2_Resistor_SMD:R_0603, symbol V2_Device:R_0603_2k7
- removed R107, R114: 5k1, V2_Resistor_SMD:R_0603, symbol V2_Device:R_0603_5k1
- removed R113: 0R005, V2_Resistor_SMD:R_1210, symbol V2_Device:R_1210_0R005
- removed TP101, TP102, TP103: ~, V2_TestPoint:TestPoint_THTPad_D1.0mm_Drill0.5mm, symbol V2_Connector:TestPoint_1.0mm_Drill0.5mm
- removed U101: CYPD3176-24LQ, V2_Package_DFN_QFN:QFN-24-1EP_4x4mm_P0.5mm_EP2.75x2.75mm, symbol V2_Interface_USB:CYPD3176-24LQ
- added C101: 10u, V2_Capacitor_SMD:C_0603, symbol V2_Device:C_0603_10u
- added C102, C103, C104: 0u1, V2_Capacitor_SMD:C_0603, symbol V2_Device:C_0603_0u1
- added C107: 10u, V2_Capacitor_SMD:C_0805, symbol V2_Device:C_0805_10u
- added C108: 1u, V2_Capacitor_SMD:C_0603, symbol V2_Device:C_0603_1u
- added D101: Orange, V2_LED:LED_0603, symbol V2_Device:LED_0603_Orange
- added D102: Red, V2_LED:LED_0603, symbol V2_Device:LED_0603_Red
- added FID101, FID102, FID103: Fiducial_Paste, V2_Fiducial:Fiducial_0.5mm_Mask1mm_Paste, symbol V2_Mechanical:Fiducial_Paste
- added INFO102: Layer_Numbers, V2_Production:Layer_Numbers, symbol V2_Production:Layer_Numbers
- added J101: 2x05_Vertical, V2_Connector_Header_1.27mm:PinHeader_2x05_P1.27mm_Vertical, symbol V2_Connector_Header_1.27mm:2x05_Vertical
- added R102, R103: 3k9, V2_Resistor_SMD:R_0603, symbol V2_Device:R_0603_3k9
- added R104, R105: 330R, V2_Resistor_SMD:R_0603, symbol V2_Device:R_0603_330R
- added TVS101, TVS102: SMBJ36CA, V2_Diode_SMD:D_SMB, symbol V2_Diode:SMBJ36CA
- added U101: CYPM1311-48LDXI, V2_Package_DFN_QFN:QFN-48-1EP_6x6mm_P0.4mm_EP4.6x4.6mm, symbol V2_Interface_USB:CYPM1311-48LDXI
- C105: renamed from C108; value 100p -> 390p; symbol V2_Device:C_0603_100p -> V2_Device:C_0603_390p; Manufacturer YAGEO -> TDK; Mouser 603-CC603JRNPO9BN101 -> 810-CGA3E2C0G1H391J; Product CC0603JRNPO9BN101 -> CGA3E2C0G1H391J080AA
- C106: renamed from C109; value 100p -> 390p; symbol V2_Device:C_0603_100p -> V2_Device:C_0603_390p; Manufacturer YAGEO -> TDK; Mouser 603-CC603JRNPO9BN101 -> 810-CGA3E2C0G1H391J; Product CC0603JRNPO9BN101 -> CGA3E2C0G1H391J080AA
- Q101, Q102: Polarity (none) -> N; Rating (none) -> 40V
- renumbered J103 to J102, J101 to J103, J102 to J104
Connections:
- net PGND is gone; now on net GND: C105.2, C106.2, J102.G (GND)
- net +1V8: now also C104.2, U101.41 (VCCD)
- net +3V3: now also R101.2, C101.1, C102.1, C103.1, D101.2 (A), D102.2 (A), J101.1 (Pin_1), R102.2, R103.2, U101.23 (VDDIO), U101.42 (VDDIO), U101.43 (VDDD), U101.5 (VDDA)
- net +VBUS: now also Q101.1 (S), C107.1, TVS101.2 (A), U101.24 (VBUS_IN_NGDO), U101.31 (VBUS_C); no longer Q101.5 (D), R101.1
- net +VLINK: now also Q102.1 (S), C108.1, TVS102.2 (A), U101.25 (VBUS_OUT_NGDO); no longer Q102.5 (D)
- net GND: now also C101.2, C102.2, C103.2, C104.1, C107.2, C108.2, J101.3 (Pin_3), TVS101.1 (K), TVS102.1 (K), U101.32 (VSS), U101.44 (VSS), U101.49 (PAD), U101.6 (VSS)
- net SCK: now also J101.4 (Pin_4), R102.1, U101.34 (P4.0/I2C_SCL)
- net SDA: now also J101.6 (Pin_6), R103.1, U101.35 (P4.1/I2C_SDA)
- net USB+: now also U101.39 (USB+)
- net USB-: now also U101.40 (USB-)
- net USB-CC1: now also U101.28 (CC1)
- net USB-CC2: now also U101.30 (CC2)
- removed net Gate: Q101.4 (G), Q102.4 (G), R101.2
- removed net Source: Q101.1 (S), Q102.1 (S)
- new net: D102.1 (K), R105.1
- new net: D101.1 (K), R104.1
- new net Drain: Q101.5 (D), Q102.5 (D)
- new net LED-Orange: R104.2, U101.11 (P5.5)
- new net LED-Red: R105.2, U101.10 (P5.3)
- new net RESET: J101.5 (Pin_5), R101.1, U101.33 (XRES)
- new net Rail-Input: Q101.4 (G), U101.27 (VBUS_IN_CTRL)
- new net Rail-Output: Q102.4 (G), U101.26 (VBUS_OUT_CTRL)
- new net SWCLK: J101.7 (Pin_7), U101.12 (P1.1/SWD_CLK)
- new net SWDIO: J101.9 (Pin_9), U101.13 (P1.2/SWD_IO)
- new net UART-RX: J101.8 (Pin_8), U101.3 (P3.5/UART_RX)
- new net UART-TX: J101.10 (Pin_10), U101.4 (P3.6/UART_TX)
- no-connect marks 5 -> 25
Other:
- note added: "Infineon / Cypress KitProg3"
- note removed: "0A"
- note removed: "1A"
- note removed: "20V"
- note removed: "9-20V, Minimum 1A"
- note removed: "9V"
- note removed: "Current Sensing The power return path between PGND and GND"
- moved on the sheet: C105, C106, ICON101, INFO101, J102, J103, J104

Commit message: Refresh
Parts:
- TVS101, TVS102: value SMBJ36CA -> SMBJ33CA; symbol V2_Diode:SMBJ36CA -> V2_Diode:SMBJ33CA; Mouser 652-SMBJ36CA-Q -> 652-SMBJ33CA-Q; Product SMBJ36CA-Q -> SMBJ33CA-Q; Rating 36V -> 33V

Commit message: Update library
Parts:
- removed J101: 2x05_Vertical, V2_Connector_Header_1.27mm:PinHeader_2x05_P1.27mm_Vertical, symbol V2_Connector_Header_1.27mm:2x05_Vertical
- added J1: KitProg3, V2_Connector_Debug:KitProg3, symbol V2_Connector_Debug:KitProg3
Connections:
- net +3V3: now also J1.1 (VDDD)
- net GND: now also J1.3 (GND)
- net RESET: now also J1.5 (RESET)
- net SCK: now also J1.4 (SCL)
- net SDA: now also J1.6 (SDA)
- net SWCLK: now also J1.7 (SWCLK)
- net SWDIO: now also J1.9 (SWDIO)
- net UART-RX: now also J1.8 (RX)
- net UART-TX: now also J1.10 (TX)
- no-connect marks 25 -> 24
Other:
- note removed: "Infineon / Cypress KitProg3"
