File: power-speakon/power-speakon.kicad_sch (KiCad schematic)
At the start: 11 parts, among them J101 NL4MDXX-V-3, J102 NL4MDXX-V-3, J103 WAGO 2601-1101, J104 WAGO 2601-1101

Commit message: Update Library
Parts:
- INFO101: value (none) -> ~
Changed lines of the file:
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@@
 		(dnp no)
 		(fields_autoplaced yes)
-		(property "Reference" "#PWR0102"
+		(property "Reference" "#PWR102"
 			(at 147.32 59.69 0)
 			(effects
@@
 			(project "power-speakon"
 				(path "/6c8448b4-b04d-47e1-934e-e40cbe27a7be"
-					(reference "#PWR0102")
+					(reference "#PWR102")
 					(unit 1)
 				)
@@
 		(on_board yes)
 		(dnp no)
-		(property "Reference" "#PWR0106"
+		(property "Reference" "#PWR106"
 			(at 135.89 124.46 0)
 			(effects
@@
 			(project "power-speakon"
 				(path "/6c8448b4-b04d-47e1-934e-e40cbe27a7be"
-					(reference "#PWR0106")
+					(reference "#PWR106")
 					(unit 1)
 				)
@@
 		(dnp no)
 		(fields_autoplaced yes)
-		(property "Reference" "#PWR0105"
+		(property "Reference" "#PWR105"
 			(at 167.64 110.49 0)
 			(effects
@@
 			(project "power-speakon"
 				(path "/6c8448b4-b04d-47e1-934e-e40cbe27a7be"
-					(reference "#PWR0105")
+					(reference "#PWR105")
 					(unit 1)
 				)
@@
 		(dnp no)
 		(fields_autoplaced yes)
-		(property "Reference" "#PWR0104"
+		(property "Reference" "#PWR104"
 			(at 157.48 99.06 0)
 			(effects
@@
 			(project "cover"
 				(path "/6c8448b4-b04d-47e1-934e-e40cbe27a7be"
-					(reference "#PWR0104")
+					(reference "#PWR104")
 					(unit 1)
 				)
@@
 		(on_board yes)
 		(dnp no)
-		(property "Reference" "#PWR0103"
+		(property "Reference" "#PWR103"
 			(at 147.32 95.25 0)
 			(effects
@@
 			(project "test"
 				(path "/6c8448b4-b04d-47e1-934e-e40cbe27a7be"
-					(reference "#PWR0103")
+					(reference "#PWR103")
 					(unit 1)
 				)
@@
 		(on_board yes)
 		(dnp no)
-		(property "Reference" "#FLG0102"
+		(property "Reference" "#FLG102"
 			(at 151.13 97.155 0)
 			(effects
@@
 			(project ""
 				(path "/6c8448b4-b04d-47e1-934e-e40cbe27a7be"
-					(reference "#FLG0102")
+					(reference "#FLG102")
 					(unit 1)
 				)
@@
 			)
 		)
-		(property "Value" ""
+		(property "Value" "~"
 			(at 214.63 181.61 0)
 			(effects
@@
 		(on_board yes)
 		(dnp no)
-		(property "Reference" "#FLG0101"
+		(property "Reference" "#FLG101"
 			(at 151.13 93.345 0)
 			(effects
@@
 			(project "test"
 				(path "/6c8448b4-b04d-47e1-934e-e40cbe27a7be"
-					(reference "#FLG0101")
+					(reference "#FLG101")
 					(unit 1)
 				)
@@
 		(on_board yes)
 		(dnp no)
-		(property "Reference" "#PWR0107"
+		(property "Reference" "#PWR107"
 			(at 143.51 147.32 0)
 			(effects
@@
 			(project "power-speakon"
 				(path "/6c8448b4-b04d-47e1-934e-e40cbe27a7be"
-					(reference "#PWR0107")
+					(reference "#PWR107")
 					(unit 1)
 				)
@@
 		(on_board yes)
 		(dnp no)
-		(property "Reference" "#PWR0108"
+		(property "Reference" "#PWR108"
 			(at 133.35 154.94 0)
 			(effects
@@
 			(project "power-speakon"
 				(path "/6c8448b4-b04d-47e1-934e-e40cbe27a7be"
-					(reference "#PWR0108")
+					(reference "#PWR108")
 					(unit 1)
 				)
@@
 		(dnp no)
 		(fields_autoplaced yes)
-		(property "Reference" "#PWR0101"
+		(property "Reference" "#PWR101"
 			(at 116.84 59.69 0)
 			(effects
@@
 			(project "power-speakon"
 				(path "/6c8448b4-b04d-47e1-934e-e40cbe27a7be"
-					(reference "#PWR0101")
-					(unit 1)
-				)
+					(reference "#PWR101")
+					(unit 1)
+				)

Commit message: Export stencil
Parts:
- INFO101: value ~ -> (none)
Changed lines of the file:
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@@
 	(title_block
 		(title "V2 Power SpeakOn")
-		(date "2026-02-10")
+		(date "2026-02-25")
 		(rev "2026-01-12")
 		(company "Versio Duo")
@@
 			)
 		)
-		(property "Value" "~"
+		(property "Value" ""
 			(at 214.63 181.61 0)
 			(effects
