File: power-speakon/power-speakon.kicad_sch (KiCad schematic)
At the start: 11 parts, among them J101 NL4MDXX-V-3, J102 NL4MDXX-V-3, J103 WAGO 2601-1101, J104 WAGO 2601-1101

Commit message: Update
Parts:
- J101: Id (none) -> SpeakOn:${SYMBOL_NAME}
- J102: renamed from J103; Id (none) -> WAGO:${SYMBOL_NAME}; Rating (none) -> 17.5A
- J103: renamed from J104; Id (none) -> WAGO:${SYMBOL_NAME}; Rating (none) -> 17.5A
- J104: renamed from J102; Id (none) -> SpeakOn:${SYMBOL_NAME}
- TVS101: Id (none) -> Diode:${SYMBOL_NAME}

Commit message: Refresh
Other:
- moved on the sheet: INFO101, J103
Changed lines of the file:
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@@
 	(title_block
 		(title "V2 Power SpeakOn")
-		(date "2026-04-14")
+		(date "2026-06-06")
 		(rev "2026-01-12")
 		(company "Versio Duo")
@@
 		(in_pos_files no)
 		(dnp no)
-		(fields_autoplaced yes)
 		(property "Reference" "#PWR108"
 			(at 167.64 110.49 0)
@@
 		)
 		(property "Value" "+28V"
-			(at 175.26 110.4899 90)
-			(show_name no)
-			(do_not_autoplace no)
-			(effects
-				(font
-					(size 1.27 1.27)
-				)
-				(justify left)
+			(at 178.816 110.2359 90)
+			(show_name no)
+			(do_not_autoplace no)
+			(effects
+				(font
+					(size 1.27 1.27)
+					(color 255 92 187 1)
+				)
 			)
 		)
@@
 		)
 		(property "Value" "+28V"
-			(at 159.004 95.25 90)
-			(show_name no)
-			(do_not_autoplace no)
-			(effects
-				(font
-					(size 1.27 1.27)
+			(at 159.004 95.25 0)
+			(show_name no)
+			(do_not_autoplace no)
+			(effects
+				(font
+					(size 1.27 1.27)
+					(color 255 92 187 1)
 				)
 			)
@@
 		)
 		(property "Value" "WAGO 2601-1101"
-			(at 154.94 150.368 0)
+			(at 161.798 147.32 0)
 			(show_name no)
 			(do_not_autoplace no)
@@
 	(symbol
 		(lib_id "V2_Production:Revision")
-		(at 214.63 179.07 0)
+		(at 209.55 179.07 0)
 		(unit 1)
 		(body_style 1)
@@
 		(dnp no)
 		(property "Reference" "INFO101"
-			(at 214.63 175.26 0)
+			(at 209.55 175.26 0)
 			(show_name no)
 			(do_not_autoplace no)
@@
 		)
 		(property "Value" ""
-			(at 214.63 181.61 0)
+			(at 209.55 181.61 0)
 			(hide yes)
 			(show_name no)
@@
 		)
 		(property "Footprint" "V2_Production:Revision"
-			(at 214.63 184.15 0)
+			(at 209.55 184.15 0)
 			(hide yes)
 			(show_name no)
@@
 		)
 		(property "Datasheet" ""
-			(at 214.63 179.07 0)
+			(at 209.55 179.07 0)
 			(hide yes)
 			(show_name no)
@@
 		)
 		(property "Description" ""
-			(at 214.63 179.07 0)
+			(at 209.55 179.07 0)
 			(hide yes)
 			(show_name no)
@@
 	(symbol
 		(lib_id "V2_Connector_WAGO:2601-1101")
-		(at 144.78 154.94 0)
+		(at 144.78 151.13 0)
 		(unit 1)
 		(body_style 1)
@@
 		(dnp no)
 		(property "Reference" "J103"
-			(at 146.05 154.9399 0)
+			(at 146.05 151.1299 0)
 			(show_name no)
 			(do_not_autoplace no)
@@
 		)
 		(property "Value" "WAGO 2601-1101"
-			(at 155.194 157.988 0)
+			(at 162.052 151.13 0)
 			(show_name no)
 			(do_not_autoplace no)
@@
 		)
 		(property "Footprint" "V2_Connector_WAGO:2601-1101"
-			(at 144.526 157.48 0)
+			(at 144.526 153.67 0)
 			(hide yes)
 			(show_name no)
@@
 		)
 		(property "Datasheet" ""
-			(at 144.78 158.75 0)
+			(at 144.78 154.94 0)
 			(hide yes)
 			(show_name no)
@@
 		)
 		(property "Description" ""
-			(at 144.78 154.94 0)
+			(at 144.78 151.13 0)
 			(hide yes)
 			(show_name no)
@@
 		)
 		(property "Manufacturer" "WAGO"
-			(at 144.78 166.37 0)
+			(at 144.78 162.56 0)
 			(hide yes)
 			(show_name no)
@@
 		)
 		(property "Product" "2601-1101"
-			(at 144.78 169.418 0)
+			(at 144.78 165.608 0)
 			(hide yes)
 			(show_name no)
@@
 		)
 		(property "Id" "WAGO:${SYMBOL_NAME}"
-			(at 144.78 163.83 0)
+			(at 144.78 160.02 0)
 			(hide yes)
 			(show_name no)
@@
 		)
 		(property "Rating" "17.5A"
-			(at 144.78 173.99 0)
+			(at 144.78 170.18 0)
 			(hide yes)
 			(show_name no)
@@
 		)
 		(property "Value" "+28V"
-			(at 132.842 147.066 90)
-			(show_name no)
-			(do_not_autoplace no)
-			(effects
-				(font
-					(size 1.27 1.27)
+			(at 132.588 147.066 90)
+			(show_name no)
+			(do_not_autoplace no)
+			(effects
+				(font
+					(size 1.27 1.27)
+					(color 255 92 187 1)
 				)
 			)
@@
 	(symbol
 		(lib_id "V2_power:GND")
-		(at 139.7 154.94 270)
+		(at 139.7 151.13 270)
 		(unit 1)
 		(body_style 1)
@@
 		(dnp no)
 		(property "Reference" "#PWR104"
-			(at 133.35 154.94 0)
+			(at 133.35 151.13 0)
 			(hide yes)
 			(show_name no)
@@
 		)
 		(property "Value" "GND"
-			(at 134.62 154.94 90)
+			(at 134.62 151.13 90)
 			(hide yes)
 			(show_name no)
@@
 		)
 		(property "Footprint" ""
-			(at 139.7 154.94 0)
+			(at 139.7 151.13 0)
 			(hide yes)
 			(show_name no)
@@
 		)
 		(property "Datasheet" ""
-			(at 139.7 154.94 0)
+			(at 139.7 151.13 0)
 			(hide yes)
 			(show_name no)
@@
 		)
 		(property "Description" ""
-			(at 129.286 154.686 0)
-			(hide yes)
-			(show_name no)
+			(at 129.286 150.876 0)
+			(hide yes)
+			(show_name no)
