File: power-speakon/power-speakon.kicad_pcb (KiCad board)
At the start: 4 copper layers, 65 x 24 mm, 18 parts, among them J101 NL4MDXX-V-3, J102 NL4MDXX-V-3, J103 WAGO 2601-1101, J104 WAGO 2601-1101, Q201 BSC010N04LS, Q202 BSC010N04LS, U201 LM74502-Q1

Commit message: Export stencil
Changed lines of the file:
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@@
 	(paper "A4")
 	(title_block
-		(date "2026-02-12")
+		(date "2026-02-25")
 		(rev "2026-01-12")
 	)
@@
 			)
 		)
-		(property "Description" "Transient Voltage Suppressor Diode, Bidirectional, 36.7-40.6V"
+		(property "Description" ""
 			(at 0 0 90)
 			(unlocked yes)
@@
 			)
 		)
-		(property "Description" "Unpolarized capacitor, small symbol"
+		(property "Description" ""
 			(at 0 0 90)
 			(layer "F.Fab")
@@
 			)
 		)
-		(property "Description" "Fiducial Marker"
+		(property "Description" ""
 			(at 0 0 0)
 			(unlocked yes)
@@
 			)
 		)
-		(property "Description" "Resistor, small symbol"
+		(property "Description" ""
 			(at 0 0 90)
 			(layer "F.Fab")
@@
 			)
 		)
-		(property "Description" "Fiducial Marker"
+		(property "Description" ""
 			(at 0 0 0)
 			(unlocked yes)
@@
 			)
 		)
-		(property "Description" "Reverse Polarity Protection Controller"
+		(property "Description" ""
 			(at 0 0 270)
 			(unlocked yes)
@@
 			)
 		)
-		(property "Description" "Unpolarized capacitor, small symbol"
+		(property "Description" ""
 			(at 0 0 90)
 			(layer "F.Fab")
@@
 			)
 		)
-		(property "Description" "Resistor, small symbol"
+		(property "Description" ""
 			(at 0 0 270)
 			(layer "F.Fab")
@@
 			)
 		)
-		(property "Description" "Fiducial Marker"
+		(property "Description" ""
 			(at 0 0 0)
 			(unlocked yes)
@@
 			)
 		)
-		(property "Datasheet" "https://www.neutrik.com/en/product/nl4mdxx-v-3"
+		(property "Datasheet" ""
 			(at -0.7 3.6 0)
 			(unlocked yes)
@@
 			)
 		)
-		(property "Description" "speakON Chassis Connectors, 4 pole chassis connector, grey D-size flange, self tapping screw holes (A-screw), vertical PCB mount. Replaces NL4MD-V-1"
+		(property "Description" ""
 			(at -0.7 3.6 0)
 			(unlocked yes)
@@
 			)
 		)
-		(property "Datasheet" "https://www.neutrik.com/en/product/nl4mdxx-v-3"
+		(property "Datasheet" ""
 			(at -0.7 3.6 0)
 			(unlocked yes)
@@
 			)
 		)
-		(property "Description" "speakON Chassis Connectors, 4 pole chassis connector, grey D-size flange, self tapping screw holes (A-screw), vertical PCB mount. Replaces NL4MD-V-1"
+		(property "Description" ""
 			(at -0.7 3.6 0)
 			(unlocked yes)

Commit message: Update
Parts:
- renumbered J103 to J102, J104 to J103, J102 to J104

Commit message: Refresh
Parts:
- C201, C202: footprint V2_Capacitor_SMD:C_0603 -> V2_Capacitor_SMD:C_1608
- R201, R202: footprint V2_Resistor_SMD:R_0603 -> V2_Resistor_SMD:R_1608
Changed lines of the file:
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@@
 	(paper "A4")
 	(title_block
-		(date "2026-02-25")
+		(date "2026-06-06")
 		(rev "2026-01-12")
 	)
@@
 		)
 	)
-	(footprint "V2_Capacitor_SMD:C_0603"
+	(footprint "V2_Capacitor_SMD:C_1608"
 		(layer "F.Cu")
 		(at 152.25 83.25 90)
-		(descr "Capacitor SMD 0603 (1608 Metric), square (rectangular) end terminal, IPC-7351 nominal, (Body size source: IPC-SM-782 page 76, https://www.pcb-3d.com/wordpress/wp-content/uploads/ipc-sm-782a_amendment_1_and_2.pdf), generated with kicad-footprint-generator")
 		(tags "capacitor")
 		(property "Reference" "C201"
@@
 			)
 		)
-		(property "Id" "Capacitor:0603_0u1"
+		(property "Id" "Capacitor:1608_0u1"
 			(at 0 0 90)
 			(unlocked yes)
@@
 		)
 		(embedded_fonts no)
-		(model "../../3dmodels/V2_Capacitor_SMD.3dshapes/C_0603_1608Metric.step"
+		(model "../../3dmodels/V2_Capacitor_SMD.3dshapes/C_1608.step"
 			(offset
 				(xyz 0 0 0)
@@
 			)
 			(rotate
-				(xyz 0 0 0)
+				(xyz -0 -0 -0)
 			)
 		)
@@
 		(embedded_fonts no)
 	)
-	(footprint "V2_Resistor_SMD:R_0603"
+	(footprint "V2_Resistor_SMD:R_1608"
 		(layer "F.Cu")
 		(at 160.75 83.25 90)
-		(descr "Resistor SMD 0603 (1608 Metric), square (rectangular) end terminal, IPC-7351 nominal, (Body size source: IPC-SM-782 page 72, https://www.pcb-3d.com/wordpress/wp-content/uploads/ipc-sm-782a_amendment_1_and_2.pdf), generated with kicad-footprint-generator")
 		(tags "resistor")
 		(property "Reference" "R202"
@@
 			)
 		)
-		(property "Id" "Resistor:0603_3k9"
+		(property "Id" "Resistor:1608_3k9"
 			(at 0 0 90)
 			(unlocked yes)
@@
 		)
 		(embedded_fonts no)
-		(model "../../3dmodels/V2_Resistor_SMD.3dshapes/R_0603_1608Metric.step"
+		(model "../../3dmodels/V2_Resistor_SMD.3dshapes/R_1608.step"
 			(offset
 				(xyz 0 0 0)
@@
 		)
 	)
-	(footprint "V2_Capacitor_SMD:C_0603"
+	(footprint "V2_Capacitor_SMD:C_1608"
 		(layer "F.Cu")
 		(at 153.75 83.25 90)
-		(descr "Capacitor SMD 0603 (1608 Metric), square (rectangular) end terminal, IPC-7351 nominal, (Body size source: IPC-SM-782 page 76, https://www.pcb-3d.com/wordpress/wp-content/uploads/ipc-sm-782a_amendment_1_and_2.pdf), generated with kicad-footprint-generator")
 		(tags "capacitor")
 		(property "Reference" "C202"
@@
 			)
 		)
-		(property "Id" "Capacitor:0603_0u22"
+		(property "Id" "Capacitor:1608_0u22"
 			(at 0 0 90)
 			(unlocked yes)
@@
 		)
 		(embedded_fonts no)
-		(model "../../3dmodels/V2_Capacitor_SMD.3dshapes/C_0603_1608Metric.step"
+		(model "../../3dmodels/V2_Capacitor_SMD.3dshapes/C_1608.step"
 			(offset
 				(xyz 0 0 0)
@@
 			)
 			(rotate
-				(xyz 0 0 0)
+				(xyz -0 -0 -0)
 			)
 		)
 	)
-	(footprint "V2_Resistor_SMD:R_0603"
+	(footprint "V2_Resistor_SMD:R_1608"
 		(layer "F.Cu")
 		(at 159.25 83.25 -90)
-		(descr "Resistor SMD 0603 (1608 Metric), square (rectangular) end terminal, IPC-7351 nominal, (Body size source: IPC-SM-782 page 72, https://www.pcb-3d.com/wordpress/wp-content/uploads/ipc-sm-782a_amendment_1_and_2.pdf), generated with kicad-footprint-generator")
 		(tags "resistor")
 		(property "Reference" "R201"
@@
 			)
 		)
-		(property "Id" "Resistor:0603_100k"
+		(property "Id" "Resistor:1608_100k"
 			(at 0 0 270)
 			(unlocked yes)
@@
 		)
 		(embedded_fonts no)
-		(model "../../3dmodels/V2_Resistor_SMD.3dshapes/R_0603_1608Metric.step"
+		(model "../../3dmodels/V2_Resistor_SMD.3dshapes/R_1608.step"
 			(offset
 				(xyz 0 0 0)
@@
 			(remove_unused_layers yes)
 			(keep_end_layers yes)
-			(zone_layer_connections)
+			(zone_layer_connections "In1.Cu" "In2.Cu")
 			(net "GND")
 			(pinfunction "1-_1-")
@@
 			(remove_unused_layers yes)
 			(keep_end_layers yes)
-			(zone_layer_connections)
+			(zone_layer_connections "In1.Cu" "In2.Cu")
 			(net "GND")
 			(pinfunction "1-_1-")
@@
 			(remove_unused_layers yes)
 			(keep_end_layers yes)
-			(zone_layer_connections)
+			(zone_layer_connections "In1.Cu" "In2.Cu")
 			(net "GND")
 			(pintype "passive")
@@
 			(remove_unused_layers yes)
 			(keep_end_layers yes)
-			(zone_layer_connections)
+			(zone_layer_connections "In1.Cu" "In2.Cu")
 			(net "GND")
 			(pintype "passive")
@@
 	)
 	(segment
-		(start 154.1125 82.1125)
-		(end 155.525 82.1125)
+		(start 159.25 84.075)
+		(end 159.075 84.075)
 		(width 0.2)
 		(layer "F.Cu")
-		(net "Net-(U201-VCAP)")
+		(net "/Polarity Protection/Overvoltage")
 	)
 	(segment
-		(start 153.75 82.475)
-		(end 154.1125 82.1125)
+		(start 159.075 84.075)
+		(end 158.5 83.5)
 		(width 0.2)
 		(layer "F.Cu")
-		(net "Net-(U201-VCAP)")
+		(net "/Polarity Protection/Overvoltage")
+	)
+	(segment
+		(start 156.825 83.675)
+		(end 156.825 84.3875)
+		(width 0.2)
+		(layer "F.Cu")
+		(net "/Polarity Protection/Overvoltage")
+	)
+	(segment
+		(start 158.5 83.5)
+		(end 157 83.5)
+		(width 0.2)
+		(layer "F.Cu")
+		(net "/Polarity Protection/Overvoltage")
+	)
+	(segment
+		(start 157 83.5)
+		(end 156.825 83.675)
+		(width 0.2)
+		(layer "F.Cu")
+		(net "/Polarity Protection/Overvoltage")
+	)
+	(segment
+		(start 160.75 84.075)
+		(end 159.25 84.075)
+		(width 0.2)
+		(layer "F.Cu")
+		(net "/Polarity Protection/Overvoltage")
 	)
 	(segment
@@
 	)
 	(segment
-		(start 159.25 84.075)
-		(end 159.075 84.075)
-		(width 0.2)
-		(layer "F.Cu")
-		(net "/Polarity Protection/Overvoltage")
-	)
-	(segment
-		(start 159.075 84.075)
-		(end 158.5 83.5)
-		(width 0.2)
-		(layer "F.Cu")
-		(net "/Polarity Protection/Overvoltage")
-	)
-	(segment
-		(start 156.825 83.675)
-		(end 156.825 84.3875)
-		(width 0.2)
-		(layer "F.Cu")
-		(net "/Polarity Protection/Overvoltage")
-	)
-	(segment
-		(start 158.5 83.5)
-		(end 157 83.5)
-		(width 0.2)
-		(layer "F.Cu")
-		(net "/Polarity Protection/Overvoltage")
-	)
-	(segment
-		(start 157 83.5)
-		(end 156.825 83.675)
+		(start 154.1125 82.1125)
+		(end 155.525 82.1125)
 		(width 0.2)
 		(layer "F.Cu")
-		(net "/Polarity Protection/Overvoltage")
+		(net "Net-(U201-VCAP)")
 	)
 	(segment
-		(start 160.75 84.075)
-		(end 159.25 84.075)
+		(start 153.75 82.475)
+		(end 154.1125 82.1125)
 		(width 0.2)
 		(layer "F.Cu")
-		(net "/Polarity Protection/Overvoltage")
+		(net "Net-(U201-VCAP)")
 	)
 	(zone
