File: usb/usb.kicad_sch (KiCad schematic)
At the start: 14 parts, among them J101 DX07S016JA3, J102 2x05_Horizontal

Commit message: Update
Parts:
- C101: Id (none) -> Capacitor:${SYMBOL_NAME}
- INFO102: value ~ -> (none)
- J101: Id (none) -> USB:${SYMBOL_NAME}; Rating (none) -> USB2.0
- J102: Id (none) -> Header:${SYMBOL_NAME}; Rating (none) -> 1A
- R101, R102: Id (none) -> Resistor:${SYMBOL_NAME}

Commit message: Good Bye Imperial
Parts:
- C101: footprint V2_Capacitor_SMD:C_0603 -> V2_Capacitor_SMD:C_1608; symbol V2_Capacitor:0603_0u1 -> V2_Capacitor:1608_0u1
- R101, R102: footprint V2_Resistor_SMD:R_0603 -> V2_Resistor_SMD:R_1608; symbol V2_Resistor:0603_5k1 -> V2_Resistor:1608_5k1
Changed lines of the file:
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@@
 	)
 	(symbol
-		(lib_id "V2_Resistor:0603_5k1")
+		(lib_id "V2_Resistor:1608_5k1")
 		(at 128.27 91.44 90)
 		(unit 1)
@@
 			)
 		)
-		(property "Footprint" "V2_Resistor_SMD:R_0603"
+		(property "Footprint" "V2_Resistor_SMD:R_1608"
 			(at 144.018 91.44 0)
 			(hide yes)
@@
 	)
 	(symbol
-		(lib_id "V2_Capacitor:0603_0u1")
+		(lib_id "V2_Capacitor:1608_0u1")
 		(at 154.94 101.6 0)
 		(unit 1)
@@
 			)
 		)
-		(property "Footprint" "V2_Capacitor_SMD:C_0603"
+		(property "Footprint" "V2_Capacitor_SMD:C_1608"
 			(at 154.94 118.618 0)
 			(hide yes)
@@
 	)
 	(symbol
-		(lib_id "V2_Resistor:0603_5k1")
+		(lib_id "V2_Resistor:1608_5k1")
 		(at 128.27 93.98 90)
 		(unit 1)
@@
 			)
 		)
-		(property "Footprint" "V2_Resistor_SMD:R_0603"
+		(property "Footprint" "V2_Resistor_SMD:R_1608"
 			(at 144.018 93.98 0)
 			(hide yes)

Commit message: Refresh
Parts:
- INFO102: renamed from INFO101; value Layer_Numbers -> Layer_Numbers-4; footprint V2_Production:Layer_Numbers -> V2_Production:Layer_Numbers-4; symbol V2_Production:Layer_Numbers -> V2_Production:Layer_Numbers-4
- renumbered INFO102 to INFO101
Changed lines of the file:
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@@
 	)
 	(symbol
-		(lib_id "V2_Production:Layer_Numbers")
+		(lib_id "V2_Production:Layer_Numbers-4")
 		(at 227.33 156.21 0)
 		(unit 1)
@@
 		(in_pos_files yes)
 		(dnp no)
-		(property "Reference" "INFO101"
+		(property "Reference" "INFO102"
 			(at 223.52 152.3999 0)
 			(show_name no)
@@
 			)
 		)
-		(property "Value" "Layer_Numbers"
+		(property "Value" "Layer_Numbers-4"
 			(at 222.25 152.3999 0)
 			(hide yes)
@@
 			)
 		)
-		(property "Footprint" "V2_Production:Layer_Numbers"
+		(property "Footprint" "V2_Production:Layer_Numbers-4"
 			(at 227.33 162.56 0)
 			(hide yes)
@@
 			(project "usb"
 				(path "/6c8448b4-b04d-47e1-934e-e40cbe27a7be"
-					(reference "INFO101")
+					(reference "INFO102")
 					(unit 1)
 				)
@@
 		(dnp no)
 		(fields_autoplaced yes)
-		(property "Reference" "#PWR106"
+		(property "Reference" "#PWR0108"
 			(at 137.16 93.98 0)
 			(hide yes)
@@
 			(project "usb"
 				(path "/6c8448b4-b04d-47e1-934e-e40cbe27a7be"
-					(reference "#PWR106")
+					(reference "#PWR0108")
 					(unit 1)
 				)
@@
 		(dnp no)
 		(fields_autoplaced yes)
-		(property "Reference" "#PWR105"
+		(property "Reference" "#PWR0107"
 			(at 137.16 91.44 0)
 			(hide yes)
@@
 			(project "usb"
 				(path "/6c8448b4-b04d-47e1-934e-e40cbe27a7be"
-					(reference "#PWR105")
+					(reference "#PWR0107")
 					(unit 1)
 				)
@@
 		(in_pos_files no)
 		(dnp no)
-		(property "Reference" "#PWR111"
+		(property "Reference" "#PWR0112"
 			(at 207.01 106.68 0)
 			(hide yes)
@@
 		)
 		(property "Value" "+VBUS"
-			(at 197.104 106.68 90)
-			(show_name no)
-			(do_not_autoplace no)
-			(effects
-				(font
-					(size 1.27 1.27)
+			(at 197.104 106.68 0)
+			(show_name no)
+			(do_not_autoplace no)
+			(effects
+				(font
+					(size 1.27 1.27)
+					(color 255 92 187 1)
 				)
 			)
@@
 			(project "usb"
 				(path "/6c8448b4-b04d-47e1-934e-e40cbe27a7be"
-					(reference "#PWR111")
+					(reference "#PWR0112")
 					(unit 1)
 				)
@@
 		(in_pos_files yes)
 		(dnp no)
-		(property "Reference" "#FLG103"
+		(property "Reference" "#FLG0103"
 			(at 102.87 66.675 0)
 			(hide yes)
@@
 			(project "usb"
 				(path "/6c8448b4-b04d-47e1-934e-e40cbe27a7be"
-					(reference "#FLG103")
+					(reference "#FLG0103")
 					(unit 1)
 				)
@@
 		(in_pos_files no)
 		(dnp no)
-		(property "Reference" "#PWR107"
+		(property "Reference" "#PWR0109"
 			(at 154.94 102.87 0)
 			(hide yes)
@@
 		)
 		(property "Value" "+VBUS"
-			(at 152.4 93.98 0)
-			(show_name no)
-			(do_not_autoplace no)
-			(effects
-				(font
-					(size 1.27 1.27)
-				)
-				(justify left)
+			(at 154.94 92.71 0)
+			(show_name no)
+			(do_not_autoplace no)
+			(effects
+				(font
+					(size 1.27 1.27)
+					(color 255 92 187 1)
+				)
 			)
 		)
@@
 			(project "usb"
 				(path "/6c8448b4-b04d-47e1-934e-e40cbe27a7be"
-					(reference "#PWR107")
+					(reference "#PWR0109")
 					(unit 1)
 				)
@@
 		(in_pos_files no)
 		(dnp no)
-		(property "Reference" "#PWR113"
+		(property "Reference" "#PWR0101"
 			(at 92.71 128.27 0)
 			(hide yes)
@@
 			(project "usb"
 				(path "/6c8448b4-b04d-47e1-934e-e40cbe27a7be"
-					(reference "#PWR113")
+					(reference "#PWR0101")
 					(unit 1)
 				)
@@
 		(in_pos_files no)
 		(dnp no)
-		(fields_autoplaced yes)
-		(property "Reference" "#PWR104"
+		(property "Reference" "#PWR0106"
 			(at 109.22 86.36 0)
 			(hide yes)
@@
 		)
 		(property "Value" "+VBUS"
-			(at 116.84 86.3599 90)
-			(show_name no)
-			(do_not_autoplace no)
-			(effects
-				(font
-					(size 1.27 1.27)
-				)
-				(justify left)
+			(at 121.666 86.3599 90)
+			(show_name no)
+			(do_not_autoplace no)
+			(effects
+				(font
+					(size 1.27 1.27)
+					(color 255 92 187 1)
+				)
 			)
 		)
@@
 			(project "usb"
 				(path "/6c8448b4-b04d-47e1-934e-e40cbe27a7be"
-					(reference "#PWR104")
+					(reference "#PWR0106")
 					(unit 1)
 				)
@@
 		(in_pos_files no)
 		(dnp no)
-		(fields_autoplaced yes)
-		(property "Reference" "#PWR103"
+		(property "Reference" "#PWR0105"
 			(at 109.22 68.58 0)
 			(hide yes)
@@
 		)
 		(property "Value" "Shield"
-			(at 106.68 68.5799 90)
+			(at 108.712 68.5799 90)
 			(show_name no)
 			(do_not_autoplace no)
@@
 			(project "usb"
 				(path "/6c8448b4-b04d-47e1-934e-e40cbe27a7be"
-					(reference "#PWR103")
+					(reference "#PWR0105")
 					(unit 1)
 				)
@@
 		(dnp no)
 		(fields_autoplaced yes)
-		(property "Reference" "#PWR109"
+		(property "Reference" "#PWR0113"
 			(at 212.09 101.6 0)
 			(hide yes)
@@
 		)
 		(property "Value" "+VBUS"
-			(at 219.71 101.5999 90)
-			(show_name no)
-			(do_not_autoplace no)
-			(effects
-				(font
-					(size 1.27 1.27)
-				)
-				(justify left)
+			(at 219.71 101.5999 0)
+			(show_name no)
+			(do_not_autoplace no)
+			(effects
+				(font
+					(size 1.27 1.27)
+					(color 255 92 187 1)
+				)
 			)
 		)
@@
 			(project "usb"
 				(path "/6c8448b4-b04d-47e1-934e-e40cbe27a7be"
-					(reference "#PWR109")
+					(reference "#PWR0113")
 					(unit 1)
 				)
@@
 		(in_pos_files yes)
 		(dnp no)
-		(property "Reference" "#FLG102"
+		(property "Reference" "#FLG0102"
 			(at 102.87 61.595 0)
 			(hide yes)
@@
 			(project "usb"
 				(path "/6c8448b4-b04d-47e1-934e-e40cbe27a7be"
-					(reference "#FLG102")
+					(reference "#FLG0102")
 					(unit 1)
 				)
@@
 		(dnp no)
 		(fields_autoplaced yes)
-		(property "Reference" "#PWR114"
+		(property "Reference" "#PWR0102"
 			(at 100.33 128.27 0)
 			(hide yes)
@@
 			(project "usb"
 				(path "/6c8448b4-b04d-47e1-934e-e40cbe27a7be"
-					(reference "#PWR114")
+					(reference "#PWR0102")
 					(unit 1)
 				)
@@
 		(dnp no)
 		(fields_autoplaced yes)
-		(property "Reference" "#PWR110"
+		(property "Reference" "#PWR0110"
 			(at 154.94 110.49 0)
 			(hide yes)
@@
 			(project "usb"
 				(path "/6c8448b4-b04d-47e1-934e-e40cbe27a7be"
-					(reference "#PWR110")
+					(reference "#PWR0110")
 					(unit 1)
 				)
@@
 		(in_pos_files yes)
 		(dnp no)
-		(property "Reference" "INFO102"
+		(property "Reference" "INFO101"
 			(at 205.74 171.45 0)
 			(show_name no)
@@
 			(project "usb"
 				(path "/6c8448b4-b04d-47e1-934e-e40cbe27a7be"
-					(reference "INFO102")
+					(reference "INFO101")
 					(unit 1)
 				)
@@
 		(in_pos_files no)
 		(dnp no)
-		(fields_autoplaced yes)
-		(property "Reference" "#PWR101"
+		(property "Reference" "#PWR0103"
 			(at 99.06 58.42 0)
 			(hide yes)
@@
 		)
 		(property "Value" "+VBUS"
-			(at 106.68 58.4199 90)
-			(show_name no)
-			(do_not_autoplace no)
-			(effects
-				(font
-					(size 1.27 1.27)
-				)
-				(justify left)
+			(at 112.268 58.6739 90)
+			(show_name no)
+			(do_not_autoplace no)
+			(effects
+				(font
+					(size 1.27 1.27)
+					(color 255 92 187 1)
+				)
 			)
 		)
@@
 			(project "usb"
 				(path "/6c8448b4-b04d-47e1-934e-e40cbe27a7be"
-					(reference "#PWR101")
+					(reference "#PWR0103")
 					(unit 1)
 				)
@@
 		(in_pos_files yes)
 		(dnp no)
-		(property "Reference" "#PWR112"
+		(property "Reference" "#PWR0114"
 			(at 222.25 106.68 0)
 			(hide yes)
@@
 			(project "usb"
 				(path "/6c8448b4-b04d-47e1-934e-e40cbe27a7be"
-					(reference "#PWR112")
+					(reference "#PWR0114")
 					(unit 1)
 				)
@@
 		(in_pos_files yes)
 		(dnp no)
-		(property "Reference" "#PWR108"
+		(property "Reference" "#PWR0111"
 			(at 196.85 101.6 0)
 			(hide yes)
@@
 			(project "usb"
 				(path "/6c8448b4-b04d-47e1-934e-e40cbe27a7be"
-					(reference "#PWR108")
+					(reference "#PWR0111")
 					(unit 1)
 				)
@@
 		(dnp no)
 		(fields_autoplaced yes)
-		(property "Reference" "#PWR102"
+		(property "Reference" "#PWR0104"
 			(at 109.22 63.5 0)
 			(hide yes)
@@
 			(project "usb"
 				(path "/6c8448b4-b04d-47e1-934e-e40cbe27a7be"
-					(reference "#PWR102")
+					(reference "#PWR0104")
 					(unit 1)
 				)
@@
 		(in_pos_files yes)
 		(dnp no)
-		(property "Reference" "#FLG101"
+		(property "Reference" "#FLG0101"
 			(at 102.87 56.515 0)
 			(hide yes)
@@
 			(project "usb"
 				(path "/6c8448b4-b04d-47e1-934e-e40cbe27a7be"
-					(reference "#FLG101")
-					(unit 1)
-				)
+					(reference "#FLG0101")
+					(unit 1)
+				)
