File: usb/usb.kicad_pcb (KiCad board)
At the start: 4 copper layers, 45 x 17.5 mm, 14 parts, among them J101 DX07S016JA3, J102 2x05_Horizontal

Commit message: Update
Connections:
- net +VBUS renamed /+VBUS
- net Shield renamed /Shield

Commit message: Refresh
Parts:
- C101: footprint V2_Capacitor_SMD:C_0603 -> V2_Capacitor_SMD:C_1608
- INFO102: renamed from INFO101; value Layer_Numbers -> Layer_Numbers-4; footprint V2_Production:Layer_Numbers -> V2_Production:Layer_Numbers-4
- R101, R102: footprint V2_Resistor_SMD:R_0603 -> V2_Resistor_SMD:R_1608
- renumbered INFO102 to INFO101
Routing:
- net /USB+: track 30.1 -> 29.6 mm, vias 2 -> 0
- net GND: vias 29 -> 28
