File: power-link-usb/hardware/PowerDelivery.kicad_sch (KiCad schematic)
At the start: 21 parts, among them J201 DX07S016JA3, J202 KitProg3, Q201 BSC010N04LS, Q202 BSC010N04LS, U201 CYPM1311-48LDXI

Commit message: Good Bye Imperial
Parts:
- C201: footprint V2_Capacitor_SMD:C_0603 -> V2_Capacitor_SMD:C_1608; symbol V2_Capacitor:0603_10u -> V2_Capacitor:1608_10u
- C202, C204, C205: footprint V2_Capacitor_SMD:C_0603 -> V2_Capacitor_SMD:C_1608; symbol V2_Capacitor:0603_0u1 -> V2_Capacitor:1608_0u1
- C203: footprint V2_Capacitor_SMD:C_0805 -> V2_Capacitor_SMD:C_2012; symbol V2_Capacitor:0805_10u -> V2_Capacitor:2012_10u
- C206: footprint V2_Capacitor_SMD:C_0603 -> V2_Capacitor_SMD:C_1608; symbol V2_Capacitor:0603_1u -> V2_Capacitor:1608_1u
- C207, C208: footprint V2_Capacitor_SMD:C_0603 -> V2_Capacitor_SMD:C_1608; symbol V2_Capacitor:0603_390p -> V2_Capacitor:1608_390p
- D201: symbol V2_LED:0603_Orange -> V2_LED:1608_Orange
- D202: symbol V2_LED:0603_Red -> V2_LED:1608_Red
- R201: footprint V2_Resistor_SMD:R_0603 -> V2_Resistor_SMD:R_1608; symbol V2_Resistor:0603_10k -> V2_Resistor:1608_10k
- R202, R203: footprint V2_Resistor_SMD:R_0603 -> V2_Resistor_SMD:R_1608; symbol V2_Resistor:0603_3k9 -> V2_Resistor:1608_3k9
- R204, R205: footprint V2_Resistor_SMD:R_0603 -> V2_Resistor_SMD:R_1608; symbol V2_Resistor:0603_330R -> V2_Resistor:1608_330R
Changed lines of the file:
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@@
 	)
 	(symbol
-		(lib_id "V2_LED:0603_Red")
+		(lib_id "V2_LED:1608_Red")
 		(at 64.77 134.62 0)
 		(unit 1)
@@
 	)
 	(symbol
-		(lib_id "V2_Capacitor:0603_0u1")
+		(lib_id "V2_Capacitor:1608_0u1")
 		(at 134.62 67.31 0)
 		(unit 1)
@@
 			)
 		)
-		(property "Footprint" "V2_Capacitor_SMD:C_0603"
+		(property "Footprint" "V2_Capacitor_SMD:C_1608"
 			(at 134.62 84.328 0)
 			(hide yes)
@@
 	)
 	(symbol
-		(lib_id "V2_Capacitor:0603_390p")
+		(lib_id "V2_Capacitor:1608_390p")
 		(at 237.49 127 90)
 		(unit 1)
@@
 			)
 		)
-		(property "Footprint" "V2_Capacitor_SMD:C_0603"
+		(property "Footprint" "V2_Capacitor_SMD:C_1608"
 			(at 254.508 127 0)
 			(hide yes)
@@
 	)
 	(symbol
-		(lib_id "V2_Capacitor:0603_10u")
+		(lib_id "V2_Capacitor:1608_10u")
 		(at 109.22 67.31 0)
 		(unit 1)
@@
 			)
 		)
-		(property "Footprint" "V2_Capacitor_SMD:C_0603"
+		(property "Footprint" "V2_Capacitor_SMD:C_1608"
 			(at 109.22 84.328 0)
 			(hide yes)
@@
 	)
 	(symbol
-		(lib_id "V2_Resistor:0603_3k9")
+		(lib_id "V2_Resistor:1608_3k9")
 		(at 237.49 113.03 90)
 		(mirror x)
@@
 			)
 		)
-		(property "Footprint" "V2_Resistor_SMD:R_0603"
+		(property "Footprint" "V2_Resistor_SMD:R_1608"
 			(at 253.238 113.03 0)
 			(hide yes)
@@
 	)
 	(symbol
-		(lib_id "V2_Resistor:0603_330R")
+		(lib_id "V2_Resistor:1608_330R")
 		(at 55.88 134.62 270)
 		(unit 1)
@@
 			)
 		)
-		(property "Footprint" "V2_Resistor_SMD:R_0603"
+		(property "Footprint" "V2_Resistor_SMD:R_1608"
 			(at 40.132 134.62 0)
 			(hide yes)
@@
 	)
 	(symbol
-		(lib_id "V2_Capacitor:0805_10u")
+		(lib_id "V2_Capacitor:2012_10u")
 		(at 127 34.29 0)
 		(unit 1)
@@
 			)
 		)
-		(property "Footprint" "V2_Capacitor_SMD:C_0805"
+		(property "Footprint" "V2_Capacitor_SMD:C_2012"
 			(at 127 51.308 0)
 			(hide yes)
@@
 	)
 	(symbol
-		(lib_id "V2_LED:0603_Orange")
+		(lib_id "V2_LED:1608_Orange")
 		(at 64.77 123.19 0)
 		(unit 1)
@@
 	)
 	(symbol
-		(lib_id "V2_Resistor:0603_3k9")
+		(lib_id "V2_Resistor:1608_3k9")
 		(at 237.49 102.87 90)
 		(mirror x)
@@
 			)
 		)
-		(property "Footprint" "V2_Resistor_SMD:R_0603"
+		(property "Footprint" "V2_Resistor_SMD:R_1608"
 			(at 253.238 102.87 0)
 			(hide yes)
@@
 	)
 	(symbol
-		(lib_id "V2_Resistor:0603_330R")
+		(lib_id "V2_Resistor:1608_330R")
 		(at 55.88 123.19 270)
 		(unit 1)
@@
 			)
 		)
-		(property "Footprint" "V2_Resistor_SMD:R_0603"
+		(property "Footprint" "V2_Resistor_SMD:R_1608"
 			(at 40.132 123.19 0)
 			(hide yes)
@@
 	)
 	(symbol
-		(lib_id "V2_Capacitor:0603_0u1")
+		(lib_id "V2_Capacitor:1608_0u1")
 		(at 123.19 67.31 0)
 		(unit 1)
@@
 			)
 		)
-		(property "Footprint" "V2_Capacitor_SMD:C_0603"
+		(property "Footprint" "V2_Capacitor_SMD:C_1608"
 			(at 123.19 84.328 0)
 			(hide yes)
@@
 	)
 	(symbol
-		(lib_id "V2_Capacitor:0603_390p")
+		(lib_id "V2_Capacitor:1608_390p")
 		(at 237.49 138.43 90)
 		(unit 1)
@@
 			)
 		)
-		(property "Footprint" "V2_Capacitor_SMD:C_0603"
+		(property "Footprint" "V2_Capacitor_SMD:C_1608"
 			(at 254.508 138.43 0)
 			(hide yes)
@@
 	)
 	(symbol
-		(lib_id "V2_Capacitor:0603_0u1")
+		(lib_id "V2_Capacitor:1608_0u1")
 		(at 154.94 67.31 0)
 		(unit 1)
@@
 			)
 		)
-		(property "Footprint" "V2_Capacitor_SMD:C_0603"
+		(property "Footprint" "V2_Capacitor_SMD:C_1608"
 			(at 154.94 84.328 0)
 			(hide yes)
@@
 	)
 	(symbol
-		(lib_id "V2_Capacitor:0603_1u")
+		(lib_id "V2_Capacitor:1608_1u")
 		(at 166.37 34.29 0)
 		(unit 1)
@@
 			)
 		)
-		(property "Footprint" "V2_Capacitor_SMD:C_0603"
+		(property "Footprint" "V2_Capacitor_SMD:C_1608"
 			(at 166.37 51.308 0)
 			(hide yes)
@@
 	)
 	(symbol
-		(lib_id "V2_Resistor:0603_10k")
+		(lib_id "V2_Resistor:1608_10k")
 		(at 237.49 92.71 90)
 		(mirror x)
@@
 			)
 		)
-		(property "Footprint" "V2_Resistor_SMD:R_0603"
+		(property "Footprint" "V2_Resistor_SMD:R_1608"
 			(at 253.238 92.71 0)
 			(hide yes)

Commit message: Refresh
Parts:
- D201, D202: footprint V2_LED:LED_0603 -> V2_LED:LED_1608
- renumbered R204 to R201, R205 to R202, R201 to R203, R202 to R204, R203 to R205
