File: power-link-usb/hardware/power-link-usb.kicad_pcb (KiCad board)
At the start: 4 copper layers, 50 x 34.5 mm, 30 parts, among them J101 NE8FAH, J102 NE8FAH, J201 DX07S016JA3, J202 KitProg3, Q201 BSC010N04LS, Q202 BSC010N04LS, U201 CYPM1311-48LDXI

Commit message: Refresh
Parts:
- C201, C202, C204, C205, C206, C207, C208: footprint V2_Capacitor_SMD:C_0603 -> V2_Capacitor_SMD:C_1608
- C203: footprint V2_Capacitor_SMD:C_0805 -> V2_Capacitor_SMD:C_2012
- D201, D202: footprint V2_LED:LED_0603 -> V2_LED:LED_1608
- R201: renamed from R204; footprint V2_Resistor_SMD:R_0603 -> V2_Resistor_SMD:R_1608
- R202: renamed from R205; footprint V2_Resistor_SMD:R_0603 -> V2_Resistor_SMD:R_1608
- R203: renamed from R201; footprint V2_Resistor_SMD:R_0603 -> V2_Resistor_SMD:R_1608
- R204: renamed from R202; footprint V2_Resistor_SMD:R_0603 -> V2_Resistor_SMD:R_1608
- R205: renamed from R203; footprint V2_Resistor_SMD:R_0603 -> V2_Resistor_SMD:R_1608

Commit message: Refresh
Parts:
- INFO102: value Layer_Numbers -> Layer_Numbers-4; footprint V2_Production:Layer_Numbers -> V2_Production:Layer_Numbers-4
- moved INFO102 1.50 mm to (120.2, 116.2)
Routing:
- net GND: vias 64 -> 65

Commit message: Refresh
Routing:
- net /PowerDelivery/USB+: track 32.0 -> 30.7 mm
