File: power-link-usb/hardware/power-link-usb.kicad_pcb (KiCad board)
At the start: 4 copper layers, 50 x 34.5 mm, 30 parts, among them J101 NE8FAH, J102 NE8FAH, J201 DX07S016JA3, J202 KitProg3, Q201 BSC010N04LS, Q202 BSC010N04LS, U201 CYPM1311-48LDXI

Commit message: Update USB-PD
Parts:
- removed R204, R205: 3k9, V2_Resistor_SMD:R_1608
- J201: footprint V2_Connector_USB:JAE_DX07S016JA3 -> V2_Connector_USB:JAE_DX07S016JA3-PD
- J202: value KitProg3 -> Cortex; footprint V2_Connector_Debug:KitProg3 -> V2_Connector_Debug:Cortex
- moved C208 14.4 mm to (162.0, 98.5), turned to -90 degrees
- moved C207 12.3 mm to (160.5, 98.5), turned to -90 degrees
- moved R203 1.50 mm to (147.2, 89.8)
Connections:
- net /PowerDelivery/+VBUS renamed /Power USB/+VBUS
- net /PowerDelivery/+VCORE renamed /Power USB/+VCORE
- net /PowerDelivery/+VSUPPLY renamed /Power USB/+VSUPPLY
- net /PowerDelivery/Drain renamed /Power USB/Drain
- net /PowerDelivery/LED-Orange renamed /Power USB/LED-Orange
- net /PowerDelivery/LED-Red renamed /Power USB/LED-Red
- net /PowerDelivery/Rail-Input renamed /Power USB/Rail-Input
- net /PowerDelivery/Rail-Output renamed /Power USB/Rail-Output
- net /PowerDelivery/Shield renamed /Power USB/Shield
- net /PowerDelivery/USB+ renamed /Power USB/USB+
- net /PowerDelivery/USB- renamed /Power USB/USB-
- net /PowerDelivery/USB-CC1 renamed /Power USB/USB-CC1
- net /PowerDelivery/USB-CC2 renamed /Power USB/USB-CC2
- J202 pad 10: /PowerDelivery/UART-TX -> /Power USB/RESET
- J202 pad 4: /PowerDelivery/SCL -> /Power USB/SWCLK
- J202 pad 5: /PowerDelivery/RESET -> GND
- R203 pad 1: /PowerDelivery/RESET -> /Power USB/RESET
- U201 pad 12: /PowerDelivery/SWCLK -> /Power USB/SWCLK
- U201 pad 13: /PowerDelivery/SWDIO -> /Power USB/SWDIO
- U201 pad 3: /PowerDelivery/UART-RX -> /Power USB/UART-RX
- U201 pad 33: /PowerDelivery/RESET -> /Power USB/RESET
- U201 pad 34: /PowerDelivery/SCL -> unconnected-(U201-P4.0/I2C_SCL-Pad34)
- U201 pad 35: /PowerDelivery/SDA -> unconnected-(U201-P4.1/I2C_SDA-Pad35)
- U201 pad 4: /PowerDelivery/UART-TX -> /Power USB/UART-TX
Routing:
- net /Power USB/SWDIO: track 0.00 -> 27.5 mm
- net /Power USB/SWCLK: track 0.00 -> 20.9 mm
- net /PowerDelivery/SWDIO: track 17.9 -> 0.00 mm, vias 1 -> 0
- net /PowerDelivery/SDA: track 17.5 -> 0.00 mm
- net /PowerDelivery/SWCLK: track 16.4 -> 0.00 mm, vias 1 -> 0
- net /PowerDelivery/SCL: track 14.6 -> 0.00 mm, vias 2 -> 0
- net /PowerDelivery/RESET: track 14.3 -> 0.00 mm, vias 1 -> 0
- net /Power USB/RESET: track 0.00 -> 13.4 mm
- net /PowerDelivery/UART-RX: track 12.4 -> 0.00 mm
- net /PowerDelivery/UART-TX: track 11.2 -> 0.00 mm, vias 1 -> 0
- net /Power USB/+VSUPPLY: track 74.8 -> 66.3 mm, vias 8 -> 6
- net /Power USB/USB-CC1: track 33.9 -> 36.2 mm
- net /Power USB/LED-Red: track 48.2 -> 47.4 mm
- net /Power USB/LED-Orange: track 46.6 -> 45.8 mm
- net GND: track 11.4 -> 11.9 mm, vias 65 -> 64
