File: power-link-usb/hardware/power-link-usb.kicad_sch (KiCad schematic)
At the start: 9 parts, among them J101 NE8FAH, J102 NE8FAH

Commit message: Refresh
Parts:
- INFO102: value Layer_Numbers -> Layer_Numbers-4; footprint V2_Production:Layer_Numbers -> V2_Production:Layer_Numbers-4; symbol V2_Production:Layer_Numbers -> V2_Production:Layer_Numbers-4
Changed lines of the file:
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@@
 	)
 	(symbol
-		(lib_id "V2_Production:Layer_Numbers")
+		(lib_id "V2_Production:Layer_Numbers-4")
 		(at 228.6 179.07 0)
 		(unit 1)
@@
 			)
 		)
-		(property "Value" "Layer_Numbers"
+		(property "Value" "Layer_Numbers-4"
 			(at 223.52 175.2599 0)
 			(hide yes)
@@
 			)
 		)
-		(property "Footprint" "V2_Production:Layer_Numbers"
+		(property "Footprint" "V2_Production:Layer_Numbers-4"
 			(at 228.6 185.42 0)
 			(hide yes)
