File: power-link-usb/hardware/power-link-usb.kicad_sch (KiCad schematic)
At the start: 9 parts, among them J101 NE8FAH, J102 NE8FAH

Commit message: Update USB-PD
Other:
- sheet PowerDelivery renamed Power USB
- sheet Power USB: file PowerDelivery.kicad_sch -> Power-USB.kicad_sch
Changed lines of the file:
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@@
 	(title_block
 		(title "V2 Power Link USB")
-		(date "2026-06-06")
-		(rev "2026-04-08")
+		(date "2026-10-15")
+		(rev "2026-10-15")
 		(company "Versio Duo")
 		(comment 1 "USB PD for V2Link / RJ45")
@@
 			(color 255 255 194 1)
 		)
-		(property "Sheetname" "PowerDelivery"
+		(property "Sheetname" "Power USB"
 			(at 88.9 95.8084 0)
 			(show_name no)
@@
 			)
 		)
-		(property "Sheetfile" "PowerDelivery.kicad_sch"
+		(property "Sheetfile" "Power-USB.kicad_sch"
 			(at 88.9 111.0746 0)
 			(hide yes)
