File: power-link-usb/hardware/Power-USB.kicad_sch (KiCad schematic)
At the start: 21 parts, among them J201 DX07S016JA3, J202 KitProg3, Q201 BSC010N04LS, Q202 BSC010N04LS, U201 CYPM1311-48LDXI

Commit message: Update USB-PD
Parts:
- removed R204, R205: 3k9, V2_Resistor_SMD:R_1608, symbol V2_Resistor:1608_3k9
- J201: footprint V2_Connector_USB:JAE_DX07S016JA3 -> V2_Connector_USB:JAE_DX07S016JA3-PD; symbol V2_Connector_USB:JAE_DX07S016JA3 -> V2_Connector_USB:JAE_DX07S016JA3-PD
- J202: value KitProg3 -> Cortex; footprint V2_Connector_Debug:KitProg3 -> V2_Connector_Debug:Cortex; symbol V2_Connector_Debug:KitProg3 -> V2_Connector_Debug:Cortex
Connections:
- net GND: now also J202.5 (GND)
- net RESET: now also J202.10 (RESET); no longer J202.5 (RESET)
- net SWCLK: now also J202.4 (SWCLK); no longer J202.7 (SWCLK)
- net SWDIO: now also J202.2 (SWDIO); no longer J202.9 (SWDIO)
- net UART-RX: no longer J202.8 (RX)
- net UART-TX: no longer J202.10 (TX)
- net SCL: no longer names the net of U201.34 (P4.0/I2C_SCL)
- net SCL: no longer J202.4 (SCL)
- net SDA: no longer names the net of U201.35 (P4.1/I2C_SDA)
- net SDA: no longer J202.6 (SDA)
- no-connect marks 24 -> 26
