File: link-wago/link-wago.kicad_sch (KiCad schematic)
At the start: 29 parts, among them J101 WAGO 2601-1101, J102 WAGO 2601-1101, J103 NE8FAH, J104 NE8FAH, J105 2x05_Horizontal, J106 2x05_Horizontal, J107 WAGO 2065-100, J108 WAGO 2065-100, J109 WAGO 2065-100, J110 WAGO 2065-100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

Commit message: Refresh
Parts:
- INFO101: value Layer_Numbers -> Layer_Numbers-4; footprint V2_Production:Layer_Numbers -> V2_Production:Layer_Numbers-4; symbol V2_Production:Layer_Numbers -> V2_Production:Layer_Numbers-4
Connections:
- net +VBUS: no longer names the net of J111.V (VBUS)
- no-connect marks 6 -> 7
Other:
- moved on the sheet: C101, J101, J102, J107, J108, J109, J110, TVS101
