File: power-link-wago/power-link-wago.kicad_pcb (KiCad board)
At the start: 4 copper layers, 52 x 44 mm, 12 parts, among them J101 NE8FAV, J102 NE8FAV, J103 WAGO 2601-1101, J104 WAGO 2601-1101, J105 WAGO 2601-1101, J106 WAGO 2601-1101

Commit message: Fix WAGOs
Parts:
- moved ICON102 1.35 mm to (126.5, 77.2)
- moved ICON103 1.35 mm to (159.5, 77.2)
- moved J103 1.00 mm to (135.8, 81.0)
- moved J105 1.00 mm to (150.2, 81.0)
- moved J104 0.50 mm to (135.8, 77.5)
- moved J106 0.50 mm to (150.2, 77.5)
Connections:
- net +24V renamed +VLINK
Changed lines of the file:
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@@
 	(net 0 "")
 	(net 1 "GND")
-	(net 2 "+24V")
+	(net 2 "+VLINK")
 	(net 3 "/RX-A")
 	(net 4 "/TX-Z")
@@
 	(footprint "V2_Connector_WAGO:2601-1101"
 		(layer "F.Cu")
-		(at 150.25 77 90)
+		(at 150.25 77.5 90)
 		(property "Reference" "J106"
 			(at 0.1 -12 90)
@@
 			(keep_end_layers yes)
 			(zone_layer_connections "In1.Cu" "In2.Cu")
-			(net 2 "+24V")
+			(net 2 "+VLINK")
 			(pintype "passive")
 		)
@@
 			(keep_end_layers yes)
 			(zone_layer_connections "In1.Cu" "In2.Cu")
-			(net 2 "+24V")
+			(net 2 "+VLINK")
 			(pintype "passive")
 		)
@@
 	(footprint "V2_Artwork:Plus_Small"
 		(layer "F.Cu")
-		(at 125.25 76.75 90)
+		(at 126.5 77.25 90)
 		(property "Reference" "ICON102"
 			(at 0 -2.5 90)
@@
 			(keep_end_layers yes)
 			(zone_layer_connections)
-			(net 2 "+24V")
+			(net 2 "+VLINK")
 			(pintype "passive")
 		)
@@
 			(keep_end_layers yes)
 			(zone_layer_connections)
-			(net 2 "+24V")
+			(net 2 "+VLINK")
 			(pintype "passive")
 		)
@@
 	(footprint "V2_Connector_WAGO:2601-1101"
 		(layer "F.Cu")
-		(at 150.25 82 90)
+		(at 150.25 81 90)
 		(property "Reference" "J105"
 			(at 0.1 -12 90)
@@
 			(keep_end_layers yes)
 			(zone_layer_connections)
-			(net 2 "+24V")
+			(net 2 "+VLINK")
 			(pintype "passive")
 		)
@@
 			(keep_end_layers yes)
 			(zone_layer_connections)
-			(net 2 "+24V")
+			(net 2 "+VLINK")
 			(pintype "passive")
 		)
@@
 	(footprint "V2_Connector_WAGO:2601-1101"
 		(layer "F.Cu")
-		(at 135.75 82 -90)
+		(at 135.75 81 -90)
 		(property "Reference" "J103"
 			(at 0.1 -12 270)
@@
 	(footprint "V2_Connector_WAGO:2601-1101"
 		(layer "F.Cu")
-		(at 135.75 77 -90)
+		(at 135.75 77.5 -90)
 		(property "Reference" "J104"
 			(at 0.1 -12 270)
@@
 			(keep_end_layers yes)
 			(zone_layer_connections "In1.Cu" "In2.Cu")
-			(net 2 "+24V")
+			(net 2 "+VLINK")
 			(pintype "passive")
 		)
@@
 			(keep_end_layers yes)
 			(zone_layer_connections "In1.Cu" "In2.Cu")
-			(net 2 "+24V")
+			(net 2 "+VLINK")
 			(pintype "passive")
 		)
@@
 	(footprint "V2_Artwork:Plus_Small"
 		(layer "F.Cu")
-		(at 160.75 76.75)
+		(at 159.5 77.25)
 		(property "Reference" "ICON103"
 			(at 0 -2.5 0)
@@
 		(polygon
 			(pts
-				(xy 131.95 79.75) (xy 154.25 79.75) (xy 154.25 84.5) (xy 131.95 84.5)
+				(xy 131.95 79.5) (xy 154.25 79.5) (xy 154.25 83.75) (xy 131.95 83.75)
 			)
 		)
@@
 	(zone
 		(net 2)
-		(net_name "+24V")
+		(net_name "+VLINK")
 		(layers "F.Cu" "In1.Cu" "In2.Cu")
 		(hatch edge 0.5)
@@
 		(polygon
 			(pts
-				(xy 131.95 74.5) (xy 154.25 74.5) (xy 154.25 79.5) (xy 131.95 79.5)
+				(xy 131.95 74.75) (xy 154.25 74.75) (xy 154.25 79) (xy 131.95 79)
 			)
 		)
@@
 	(zone
 		(net 2)
-		(net_name "+24V")
+		(net_name "+VLINK")
 		(layer "B.Cu")
 		(hatch edge 0.5)
@@
 		(polygon
 			(pts
-				(xy 154.25 80) (xy 146.75 80) (xy 145.75 81) (xy 145.75 90.75) (xy 147.75 92.75) (xy 157 92.75)
+				(xy 154.25 79.5) (xy 146.5 79.5) (xy 145.75 80.25) (xy 145.75 90.75) (xy 147.75 92.75) (xy 157 92.75)
 				(xy 158 93.75) (xy 158 100.5) (xy 155 100.5) (xy 155 98.25) (xy 153.75 98.25) (xy 153.75 96) (xy 132 96)
 				(xy 132 101) (xy 129.25 101) (xy 129.25 98.25) (xy 127.75 98.25) (xy 127.75 93.5) (xy 128.75 92.5)
-				(xy 138.25 92.5) (xy 140.25 90.5) (xy 140.25 81) (xy 139.25 80) (xy 131.5 80) (xy 131.5 74.5) (xy 154.25 74.5)
-			)
-		)
+				(xy 138.25 92.5) (xy 140.25 90.5) (xy 140.25 80.5) (xy 139.25 79.5) (xy 131.5 79.5) (xy 131.5 75)
+				(xy 154.25 75)
+			)
+		)

Commit message: Replace Order_Number
Parts:
- H101, H102: value MountingHole_5mm -> 5mm
- INFO101: value Order_Number -> ~; footprint V2_Production:Order_Number -> V2_Production:Revision

Commit message: Refresh
Parts:
- renumbered J103 to J102, J105 to J103, J106 to J105, J102 to J106
Connections:
- net +VLINK renamed /+VLINK
- net Shield renamed /Shield
