File: power-link-wago/power-link-wago.kicad_sch (KiCad schematic)
At the start: 12 parts, among them J101 NE8FAV, J102 NE8FAV, J103 WAGO 2601-1101, J104 WAGO 2601-1101, J105 WAGO 2601-1101, J106 WAGO 2601-1101

Commit message: Refresh
Parts:
- J101: Id (none) -> EtherCon:${SYMBOL_NAME}; Rating (none) -> CAT5e
- J102: renamed from J103; Id (none) -> WAGO:${SYMBOL_NAME}; Rating (none) -> 17.5A
- J103: renamed from J105; Id (none) -> WAGO:${SYMBOL_NAME}; Rating (none) -> 17.5A
- J104: Id (none) -> WAGO:${SYMBOL_NAME}; Rating (none) -> 17.5A
- J105: renamed from J106; Id (none) -> WAGO:${SYMBOL_NAME}; Rating (none) -> 17.5A
- J106: renamed from J102; Id (none) -> EtherCon:${SYMBOL_NAME}; Rating (none) -> CAT5e
Other:
- moved on the sheet: ICON101, ICON102, ICON103, INFO101, J102, J103, J105
